File: KiCad/eth.kicad_sch (KiCad schematic)
At the start: 203 parts, among them J16 RJE361882415, J17 RJ45_LED_Shielded_x2, J18 RJ45_LED_Shielded_x2, U4 RTL8125BG-CG, U5 RTL8125BG-CG, U6 RTL8125BG-CG, U7 RTL8125BG-CG, U8 RTL8125BG-CG, Y1 25MHz, Y2 25MHz, Y3 25MHz, Y4 25MHz, Y5 25MHz

Commit message: Switch nics to i226-v
Parts:
- removed C212, C247, C257, C279: 390pF, symbol Device:C
- removed C216: 27pF, symbol Device:C_Small
- removed C242: 2.2uF, symbol Device:C_Small
- removed C268: 100nF, symbol Device:C_Small
- removed U4, U5, U6, U7, U8: RTL8125BG-CG, Package_DFN_QFN:QFN-48-1EP_6x6mm_P0.4mm_EP4.2x4.2mm, symbol custom:RTL8125BG-CG
- added C212, C257, C328, C329, C330, C331, C332, C333, C334, C335, C336, C337, C338, C339, C340, C341, C342, C346: 100nF, symbol Device:C_Small
- added C216, C242, C268, C345: 390pF, symbol Device:C
- added C247: 220nF, symbol Device:C_Small
- added C279, C343, C344: 22uF, symbol Device:C_Small
- added C347: 100pF, symbol Device:C_Small
- added L3, L4, L5, L6, L7: 1uH, symbol Device:L
- added R211: 200R, symbol Device:R_Small
- added R212, R213, R215, R216, R217, R218: 10k, symbol Device:R_Small
- added R214: 22k, symbol Device:R_Small
- added R219, R224, R225: 510R, symbol Device:R_Small
- added R220, R221, R222, R223: 75R, symbol Device:R_Small
- added U16, U18, U20, U6, U8: W25Q128JVS, Package_SO:SOIC-8_5.3x5.3mm_P1.27mm, symbol Memory_Flash:W25Q128JVS
- added U17, U19, U4, U5, U7: KTI226V, Package_DFN_QFN:QFN-56-1EP_7x7mm_P0.4mm_EP5.6x5.6mm_ThermalVias, symbol custom:KTI226V
- C171, C172, C175, C176: value 27pF -> 18pF
- C173, C174, C185, C186: value 100nF -> 220nF
- C177, C240: value 1uF -> 22uF
- C178, C254, C278: value 10uF -> 22uF
- C179, C180, C181, C190, C191, C226, C241, C252, C253, C266, C267: value 2.2uF -> 22uF
- C184, C189, C194, C197, C198, C199, C200, C205, C206, C207, C208, C223, C233, C234, C235, C238, C243, C250, C251, C265, C275, C276: value 2.2uF -> 100nF
- C187, C196, C204, C231, C249, C263: value 1uF -> 100nF
- C188, C195, C201, C202, C203, C209, C210, C232, C239, C255, C264, C277: value 10uF -> 100nF
- C192: value 100nF -> 22uF
- C214, C280: value 100pF -> 22uF
- C215, C227, C228: value 27pF -> 22uF
- C218: value 100nF -> 100pF
- C219, C272: value 1uF -> 18pF
- C220, C245, C246, C271: value 10uF -> 18pF
- C221, C222, C273, C274: value 2.2uF -> 220nF
- C244, C270: value 2.2uF -> 100pF
- C248: value 10uF -> 220nF
- C256, C258: value 100pF -> 100nF
- C259, C260: value 27pF -> 100nF
- R103, R62, R81, R86: value 75R -> 510R
- R105, R125, R126, R127, R88, R94: value 510R -> 10k
- R123, R93: value 510R -> 22k
- R124: value 510R -> 200R
- R41: value 1k -> 510R
- R42, R73, R92: value 15k -> 10k
- R43, R47, R51, R52, R54, R74, R77, R78, R79, R80, R95: value 4.7k -> 10k
- R44, R91: value 1k -> 10k
- R45: value 15k -> 200R
- R46, R49, R75, R96: value 0R -> 10k
- R48, R50, R71, R97: value 2.49k -> 10k
- R53: value 4.7k -> 22k
- R59, R60, R61, R90: value 75R -> 10k
- R65: value 1k -> 75R
- R66: value 15k -> 75R
- R67, R68: value 510R -> 75R
- R69, R98: value 4.7k -> 510R
- R70: value 0R -> 510R
- R72: value 1k -> 200R
- R76: value 2.49k -> 22k
- R89: value 75R -> 200R
- R99: value 4.7k -> 75R
Connections:
- net +3V3: now also R42.2, R43.2, R46.2, R48.2, R50.2, R59.2, R60.2, R61.2, R75.2, R92.2, R94.2, R95.2, R96.2, R97.2, R215.2, R216.2, R217.2, R218.2; no longer R123.2, R124.2, R125.2, R126.2, R52.2, R53.2, R98.2, R99.2
- net +3V3SB: now also C193.1, C194.1, C195.1, C196.1, C197.1, C198.1, C199.1, C203.1, C204.1, C205.1, C217.1, C227.2, C228.2, C229.1, C230.1, C231.1, C232.1, C233.1, C243.1, C249.2, C250.2, C251.2, C252.2, C253.2, C254.2, C255.1, C256.1, C258.1, C259.1, C269.1, C275.2, C276.2, C277.2, C278.2, C280.2, R103.2, R105.1, R125.1, R41.2, R62.2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; no longer C180.2, C181.2, C193.2, C194.2, C219.2, C220.2, C221.2, C222.2, C231.2, C232.2, C233.2, C234.2, C235.2, C236.2, C237.2, C238.2, C263.2, C264.2, C265.2, C266.2, C267.2, C269.2, C270.2, R105.2, R41.1, R43.1, R65.1, R67.2, R68.2, R69.1, R72.1, R74.1, R88.2, R91.1, R93.2, R94.2, R95.1
- net ETH0.REFCLK+: now also U4.21 (PE_CLK_P)
- net ETH0.REFCLK-: now also U4.22 (PE_CLK_N)
- net ETH0.Tx0+: now also U4.28 (PE_Rx_P)
- net ETH0.Tx0-: now also U4.27 (PE_Rx_N)
- net ETH0.~{PLTRST}: now also U4.13 (PE_RST_N)
- net ETH0.~{WAKE}: now also U4.12 (PE_WAKE_N); no longer R43.2
- net ETH1.REFCLK+: now also U5.21 (PE_CLK_P)
- net ETH1.REFCLK-: now also U5.22 (PE_CLK_N)
- net ETH1.Rx0+: now also C185.1; no longer C217.1
- net ETH1.Rx0-: now also C186.1; no longer C218.1
- net ETH1.Tx0+: now also U5.28 (PE_Rx_P)
- net ETH1.Tx0-: now also U5.27 (PE_Rx_N)
- net ETH1.~{PLTRST}: now also U5.13 (PE_RST_N)
- net ETH1.~{WAKE}: now also U5.12 (PE_WAKE_N); no longer R69.2
- net ETH2.REFCLK+: now also U7.21 (PE_CLK_P)
- net ETH2.REFCLK-: now also U7.22 (PE_CLK_N)
- net ETH2.Rx0+: now also C221.1; no longer C261.1
- net ETH2.Rx0-: now also C222.1; no longer C262.1
- net ETH2.Tx0+: now also U7.28 (PE_Rx_P)
- net ETH2.Tx0-: now also U7.27 (PE_Rx_N)
- net ETH2.~{PLTRST}: now also U7.13 (PE_RST_N)
- net ETH2.~{WAKE}: now also U7.12 (PE_WAKE_N); no longer R95.2
- net ETH3.REFCLK+: now also U17.21 (PE_CLK_P)
- net ETH3.REFCLK-: now also U17.22 (PE_CLK_N)
- net ETH3.Rx0+: now also C247.1; no longer C185.1
- net ETH3.Rx0-: now also C248.1; no longer C186.1
- net ETH3.Tx0+: now also U17.28 (PE_Rx_P)
- net ETH3.Tx0-: now also U17.27 (PE_Rx_N)
- net ETH3.~{PLTRST}: now also U17.13 (PE_RST_N)
- net ETH3.~{WAKE}: now also U17.12 (PE_WAKE_N); no longer R47.2
- net ETH4.REFCLK+: now also U19.21 (PE_CLK_P)
- net ETH4.REFCLK-: now also U19.22 (PE_CLK_N)
- net ETH4.Rx0+: now also C273.1; no longer C229.1
- net ETH4.Rx0-: now also C274.1; no longer C230.1
- net ETH4.Tx0+: now also U19.28 (PE_Rx_P)
- net ETH4.Tx0-: now also U19.27 (PE_Rx_N)
- net ETH4.~{PLTRST}: now also U19.13 (PE_RST_N)
- net ETH4.~{WAKE}: now also U19.12 (PE_WAKE_N); no longer R74.2
- net GND: now also C180.2, C181.2, C193.2, C194.2, C200.1, C201.1, C202.1, C206.1, C207.1, C208.1, C209.1, C211.1, C215.2, C217.2, C218.2, C229.2, C230.2, C231.2, C232.2, C233.2, C238.2, C245.1, C246.1, C249.1, C250.1, C251.1, C252.1, C253.1, C254.1, C259.2, C261.1, C262.1, C264.2, C265.2, C266.2, C267.2, C269.2, C270.2, C271.1, C272.1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; no longer C180.1, C181.1, C193.1, C194.1, C200.2, C201.2, C202.2, C206.2, C207.2, C208.2, C209.2, C211.2, C215.1, C221.1, C222.1, C231.1, C232.1, C233.1, C238.1, C245.2, C246.2, C248.2, C249.2, C250.2, C251.2, C252.2, C253.2, C254.2, C259.1, C264.1, C265.1, C266.1, C267.1, C269.1, C270.1, C271.2, C272.2, C273.2, C274.2, C275.2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
- net at TR4.21 (CT): now also R101.1; no longer R89.1
- net at TR4.24 (CT): now also R102.1; no longer R90.1
- net at C176.2, Y2.3: now also U5.40 (XTAL_OUT); no longer R49.1
- net at R123.1: now also U4.42 (PHY_CAL); no longer D2.2 (A)
- net at TR2.1 (CT), TR2.10 (CT), TR2.4 (CT)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: now also C216.2
- net at TR2.11 (TD4+): now also U5.54 (MDI_D_P)
- net at TR2.12 (TD4-): now also U5.55 (MDI_D_N)
- net at R59.1: now also U5.37 (SPI_CS_N/PCIE_ENA), U6.1 (~{CS}); no longer TR2.15 (CT)
- net at R60.1: now also U6.3 (~{WP}/IO_{2}); no longer TR2.18 (CT)
- net at TR2.2 (TD1+): now also U5.45 (MDI_A_P)
- net at R61.1: now also U6.7 (~{HOLD}/~{RESET}/IO_{3}); no longer TR2.21 (CT)
- net at TR2.24 (CT): now also R68.1; no longer R62.1
- net at TR2.3 (TD1-): now also U5.46 (MDI_A_N)
- net at TR2.5 (TD2+): now also U5.48 (MDI_B_P)
- net at TR2.6 (TD2-): now also U5.49 (MDI_B_N)
- net at TR2.8 (TD3+): now also U5.51 (MDI_C_P)
- net at TR2.9 (TD3-): now also U5.52 (MDI_C_N)
- net at C175.2, Y2.1: now also U5.41 (XTAL_IN)
- net at R50.1: now also U5.36 (SPI_DIN/AUX_PWR), U6.2 (DO/IO_{1})
- net at D5.1 (K): now also U17.30 (LED2)
- net at R54.1: now also U5.34 (SPI_DOUT/SEC_ENA), U6.5 (DI/IO_{0}); no longer J17.11
- net at R53.1: now also U5.42 (PHY_CAL)
- net at J17.9: now also U5.31 (LED1)
- net at C185.2: now also U5.25 (PE_Tx_P)
- net at C186.2: now also U5.24 (PE_Tx_N)
- net at TR5.1 (CT), TR5.10 (CT), TR5.4 (CT)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: now also C345.2
- net at TR5.11 (TD4+): now also U19.54 (MDI_D_P)
- net at TR5.12 (TD4-): now also U19.55 (MDI_D_N)
- net at TR5.15 (CT): now also R220.1; no longer R100.1
- net at TR5.18 (CT): now also R221.1; no longer R101.1
- net at TR5.2 (TD1+): now also U19.45 (MDI_A_P)
- net at TR5.21 (CT): now also R222.1; no longer R102.1
- net at TR5.24 (CT): now also R223.1; no longer R103.1
- net at TR5.3 (TD1-): now also U19.46 (MDI_A_N)
- net at TR5.5 (TD2+): now also U19.48 (MDI_B_P)
- net at TR5.6 (TD2-): now also U19.49 (MDI_B_N)
- net at TR5.8 (TD3+): now also U19.51 (MDI_C_P)
- net at TR5.9 (TD3-): now also U19.52 (MDI_C_N)
- net at Y5.1: now also C271.2, U19.41 (XTAL_IN); no longer C259.2
- net at Y4.1: now also C245.2, U17.41 (XTAL_IN); no longer C227.2
- net at R81.1: now also D4.2 (A); no longer TR3.15 (CT)
- net at R82.2, R83.2, R84.2: now also C244.1, R85.2; no longer C256.1, R81.2
- net at J17.24: now also R86.1; no longer R93.1
- net at R76.1: now also U7.42 (PHY_CAL)
- net at TR4.2 (TD1+): now also U17.45 (MDI_A_P)
- net at TR4.3 (TD1-): now also U17.46 (MDI_A_N)
- net at TR4.5 (TD2+): now also U17.48 (MDI_B_P)
- net at TR4.6 (TD2-): now also U17.49 (MDI_B_N)
- net at TR4.8 (TD3+): now also U17.51 (MDI_C_P)
- net at TR4.9 (TD3-): now also U17.52 (MDI_C_N)
- net at TR4.11 (TD4+): now also U17.54 (MDI_D_P)
- net at TR4.12 (TD4-): now also U17.55 (MDI_D_N)
- net at D6.1 (K): now also U19.30 (LED2)
- net at J17.23: now also U7.32 (LED0); no longer R80.1
- net at R79.1: now also U8.3 (~{WP}/IO_{2})
- net at J17.21: now also U7.31 (LED1)
- net at C262.2: now also C260.2, C261.2, C263.2, C264.1, C265.1, C266.1, C267.1, L6.1, U17.26 (VDD_VP), U17.38 (VDD_CORE), U17.44 (VDD_A), U17.50 (VDD_A), U17.56 (VDD_A), U17.9 (VDD_CORE)
- net at R70.1: now also J17.10; no longer Y3.3
- net at R100.2, R101.2, R102.2: now also C270.1, R99.2; no longer C280.1, R103.2
- net at J18.24: now also R224.1; no longer R104.1
- net at R84.1: now also TR3.21 (CT); no longer TR3.24 (CT)
- net at C171.2, Y1.1: now also U4.41 (XTAL_IN)
- net at C172.2, Y1.3: now also U4.40 (XTAL_OUT); no longer R46.1
- net at J17.22: now also R87.1; no longer R94.1
- net at R98.1: now also D5.2 (A)
- net at R48.1: now also U16.5 (DI/IO_{0}), U4.34 (SPI_DOUT/SEC_ENA)
- net at TR1.2 (TD1+): now also U4.45 (MDI_A_P)
- net at TR1.3 (TD1-): now also U4.46 (MDI_A_N)
- net at TR1.5 (TD2+): now also U4.48 (MDI_B_P)
- net at TR1.6 (TD2-): now also U4.49 (MDI_B_N)
- net at TR1.8 (TD3+): now also U4.51 (MDI_C_P)
- net at TR1.9 (TD3-): now also U4.52 (MDI_C_N)
- net at TR1.11 (TD4+): now also U4.54 (MDI_D_P)
- net at TR1.12 (TD4-): now also U4.55 (MDI_D_N)
- net at D2.1 (K): now also U4.30 (LED2)
- net at J16.D4: now also U4.32 (LED0); no longer R52.1
- net at R51.1: now also U16.2 (DO/IO_{1}), U4.36 (SPI_DIN/AUX_PWR)
- net at J16.D2: now also U4.31 (LED1)
- net at C173.2: now also U4.25 (PE_Tx_P)
- net at C174.2: now also U4.24 (PE_Tx_N)
- net at TR3.1 (CT), TR3.10 (CT), TR3.4 (CT)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: now also C242.2
- net at Y3.1: now also C219.2, U7.41 (XTAL_IN); no longer C215.2
- net at TR3.2 (TD1+): now also U7.45 (MDI_A_P)
- net at TR3.3 (TD1-): now also U7.46 (MDI_A_N)
- net at TR3.5 (TD2+): now also U7.48 (MDI_B_P)
- net at TR3.6 (TD2-): now also U7.49 (MDI_B_N)
- net at TR3.8 (TD3+): now also U7.51 (MDI_C_P)
- net at TR3.9 (TD3-): now also U7.52 (MDI_C_N)
- net at TR3.11 (TD4+): now also U7.54 (MDI_D_P)
- net at TR3.12 (TD4-): now also U7.55 (MDI_D_N)
- net at D3.1 (K): now also U5.30 (LED2)
- net at J18.11: now also U17.32 (LED0); no longer R78.1
- net at R77.1: now also U7.34 (SPI_DOUT/SEC_ENA), U8.5 (DI/IO_{0})
- net at J18.9: now also U17.31 (LED1)
- net at D3.2 (A): now also R62.1; no longer R124.1
- net at TR4.1 (CT), TR4.10 (CT), TR4.4 (CT)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: now also C268.2
- net at R97.1: now also U18.7 (~{HOLD}/~{RESET}/IO_{3})
- net at TR4.18 (CT): now also R100.1; no longer R86.1
- net at TR1.1 (CT), TR1.10 (CT), TR1.4 (CT)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: now also C211.2; no longer C211.1
- net at R67.1: now also TR2.21 (CT); no longer J17.12
- net at R99.1: now also TR4.15 (CT); no longer J18.23
- net at J18.8: now also TR4.13 (MX4-); no longer TR3.13 (MX4-)
- net at J18.7: now also TR4.14 (MX4+); no longer TR3.14 (MX4+)
- net at J18.5: now also TR4.16 (MX3-); no longer TR3.16 (MX3-)
- net at J18.4: now also TR4.17 (MX3+); no longer TR3.17 (MX3+)
- net at TR3.18 (CT): now also R83.1; no longer R82.1
- net at J18.6: now also TR4.19 (MX2-); no longer TR3.19 (MX2-)
- net at J18.3: now also TR4.20 (MX2+); no longer TR3.20 (MX2+)
- net at J18.2: now also TR4.22 (MX1-); no longer TR3.22 (MX1-)
- net at J18.1: now also TR4.23 (MX1+); no longer TR3.23 (MX1+)
- net at J18.12: now also R103.1; no longer R87.1
- net at R127.1: now also U19.36 (SPI_DIN/AUX_PWR), U20.2 (DO/IO_{1}); no longer D6.2 (A)
- net at J18.10: now also R104.1; no longer R88.1
- net at D4.1 (K): now also U7.30 (LED2)
- net at J18.21: now also U19.31 (LED1)
- net at R126.1: now also U19.35 (SPI_CLK), U20.6 (CLK); no longer D5.2 (A)
- net at R85.1: now also TR3.24 (CT); no longer TR4.15 (CT)
- net at J18.22: now also R225.1; no longer R105.1
- net at J17.20: now also TR3.13 (MX4-); no longer TR4.13 (MX4-)
- net at J17.19: now also TR3.14 (MX4+); no longer TR4.14 (MX4+)
- net at J17.17: now also TR3.16 (MX3-); no longer TR4.16 (MX3-)
- net at J17.16: now also TR3.17 (MX3+); no longer TR4.17 (MX3+)
- net at J17.18: now also TR3.19 (MX2-); no longer TR4.19 (MX2-)
- net at J17.15: now also TR3.20 (MX2+); no longer TR4.20 (MX2+)
- net at J17.14: now also TR3.22 (MX1-); no longer TR4.22 (MX1-)
- net at J17.13: now also TR3.23 (MX1+); no longer TR4.23 (MX1+)
- removed net +0V95: C195.1, C196.1, C197.1, C198.1, C199.1, C200.1, C201.1, C202.1, C203.1, C204.1, C205.1, C206.1, C207.1, C208.1, C209.1, C210.1, C239.1, C240.1, C241.1, C243.1, C244.1, C245.1, C246.1, C248.1, C249.1, C250.1, C251.1, C252.1, C253.1, C254.1, C255.1, C271.1, C272.1, C273.1, C274.1, C275.1, C276.1, C277.1, C278.1
- net ETH0.~{ISOLATE}: no longer names the net of R42.1
- net ETH0.~{ISOLATE}: now also U16.7 (~{HOLD}/~{RESET}/IO_{3}); no longer R41.2
- net ETH1.~{ISOLATE}: no longer names the net of R65.2
- net ETH1.~{ISOLATE}: now also C218.1, R66.2, R67.2, R68.2; no longer R66.1
- net ETH2.~{ISOLATE}: no longer names the net of R92.1
- net ETH2.~{ISOLATE}: now also U17.36 (SPI_DIN/AUX_PWR), U18.2 (DO/IO_{1}); no longer R91.2
- net ETH3.~{ISOLATE}: no longer names the net of R44.2
- net ETH3.~{ISOLATE}: now also U5.2 (LAN_DISABLE_N); no longer R45.1
- net ETH4.~{ISOLATE}: no longer names the net of R72.2
- net ETH4.~{ISOLATE}: now also U7.20 (RBIAS); no longer R73.1
- new net: C206.2, C207.2, C208.2, C209.2, C210.1, C212.1, C214.1, C215.1, L4.1, U5.26 (VDD_VP), U5.38 (VDD_CORE), U5.44 (VDD_A), U5.50 (VDD_A), U5.56 (VDD_A), U5.9 (VDD_CORE)
- new net: R212.2, U4.1 (LAN_PWR_GOOD)
- new net: R213.2, U4.2 (LAN_DISABLE_N)
- new net: R211.2, U4.20 (RBIAS)
- new net: C180.1, C181.1, C200.2, C201.2, C202.2, C328.2, C330.1, C331.1, L3.1, U4.26 (VDD_VP), U4.38 (VDD_CORE), U4.44 (VDD_A), U4.50 (VDD_A), U4.56 (VDD_A), U4.9 (VDD_CORE)
- new net: R52.1, U16.6 (CLK), U4.35 (SPI_CLK)
- new net: R46.1, U16.1 (~{CS}), U4.37 (SPI_CS_N/PCIE_ENA)
- new net: L3.2, U4.5 (VDD_CTRL), U4.6 (VDD_CTRL)
- new net: C234.2, C235.2, C236.2, C237.2, C238.1, C239.1, C240.1, C241.1, L5.1, U7.26 (VDD_VP), U7.38 (VDD_CORE), U7.44 (VDD_A), U7.50 (VDD_A), U7.56 (VDD_A), U7.9 (VDD_CORE)
- new net: C337.2, C338.2, C339.2, C340.2, C341.1, C342.1, C343.1, C344.1, L7.1, U19.26 (VDD_VP), U19.38 (VDD_CORE), U19.44 (VDD_A), U19.50 (VDD_A), U19.56 (VDD_A), U19.9 (VDD_CORE)
- new net: R88.2, U17.2 (LAN_DISABLE_N)
- new net: C347.1, R220.2, R221.2, R222.2, R223.2
- new net: C248.2, U17.24 (PE_Tx_N)
- new net: R45.2, U5.20 (RBIAS)
- new net: R49.1, U5.35 (SPI_CLK), U6.6 (CLK)
- new net: R216.1, U19.37 (SPI_CS_N/PCIE_ENA), U20.1 (~{CS})
- new net: R217.1, U20.3 (~{WP}/IO_{2})
- new net: R215.1, U19.34 (SPI_DOUT/SEC_ENA), U20.5 (DI/IO_{0})
- new net: R218.1, U20.7 (~{HOLD}/~{RESET}/IO_{3})
- new net: C272.2, U19.40 (XTAL_OUT), Y5.3
- new net: R90.2, U17.1 (LAN_PWR_GOOD)
- new net: R71.2, U7.2 (LAN_DISABLE_N)
- new net: D2.2 (A), R41.1
- new net: R47.2, U5.1 (LAN_PWR_GOOD)
- new net: J17.11, U5.32 (LED0)
- new net: L4.2, U5.5 (VDD_CTRL), U5.6 (VDD_CTRL)
- new net: R75.1, U7.36 (SPI_DIN/AUX_PWR), U8.2 (DO/IO_{1})
- new net: C246.2, U17.40 (XTAL_OUT), Y4.3
- new net: D6.2 (A), R219.1
- new net: R73.2, U7.1 (LAN_PWR_GOOD)
- new net: C222.2, U7.24 (PE_Tx_N)
- new net: C221.2, U7.25 (PE_Tx_P)
- new net: R74.1, U7.35 (SPI_CLK), U8.6 (CLK)
- new net: R78.1, U7.37 (SPI_CS_N/PCIE_ENA), U8.1 (~{CS})
- new net: C220.2, U7.40 (XTAL_OUT), Y3.3
- new net: L5.2, U7.5 (VDD_CTRL), U7.6 (VDD_CTRL)
- new net: R93.1, U17.42 (PHY_CAL)
- new net: R89.2, U17.20 (RBIAS)
- new net: C247.2, U17.25 (PE_Tx_P)
- new net: R94.1, U17.34 (SPI_DOUT/SEC_ENA), U18.5 (DI/IO_{0})
- new net: R91.1, U17.35 (SPI_CLK), U18.6 (CLK)
- new net: R95.1, U17.37 (SPI_CS_N/PCIE_ENA), U18.1 (~{CS})
- new net: L6.2, U17.5 (VDD_CTRL), U17.6 (VDD_CTRL)
- new net: R65.1, TR2.15 (CT)
- new net: R66.1, TR2.18 (CT)
- new net: J18.23, U19.32 (LED0)
- new net: R43.1, U16.3 (~{WP}/IO_{2})
- new net: R82.1, TR3.15 (CT)
- new net: J17.12, R69.1
- new net: R214.1, U19.42 (PHY_CAL)
- new net: R125.2, U19.1 (LAN_PWR_GOOD)
- new net: R124.2, U19.20 (RBIAS)
- new net: C274.2, U19.24 (PE_Tx_N)
- new net: R96.1, U18.3 (~{WP}/IO_{2})
- new net: R80.1, U8.7 (~{HOLD}/~{RESET}/IO_{3})
- new net: R105.2, U19.2 (LAN_DISABLE_N)
- new net: C273.2, U19.25 (PE_Tx_P)
- new net: L7.2, U19.5 (VDD_CTRL), U19.6 (VDD_CTRL)
- new net ETH0.SMBCLK: U4.11 (SMB_CLK)
- new net ETH0.SMBDAT: U4.10 (SMB_DATA), U4.4 (ULP_WAKE_N)
- new net ETH1.SMBCLK: U5.11 (SMB_CLK)
- new net ETH1.SMBDAT: U5.10 (SMB_DATA), U5.4 (ULP_WAKE_N)
- new net ETH2.SMBCLK: U7.11 (SMB_CLK)
- new net ETH2.SMBDAT: U7.10 (SMB_DATA), U7.4 (ULP_WAKE_N)
- new net ETH3.SMBCLK: U17.11 (SMB_CLK)
- new net ETH3.SMBDAT: U17.10 (SMB_DATA), U17.4 (ULP_WAKE_N)
- new net ETH4.SMBCLK: U19.11 (SMB_CLK)
- new net ETH4.SMBDAT: U19.10 (SMB_DATA), U19.4 (ULP_WAKE_N)
- no-connect marks 22 -> 35
Other:
- moved on the sheet: C171, C172, C173, C174, C211, Y1

Commit message: Work though ERC errors
Connections:
- net GND: now also J16.SH, J17.SH, J17.SH, J18.SH, J18.SH

Commit message: Re-annotate components
Parts:
- renumbered C171 to C193, C172 to C194, C245 to C195, C246 to C196, C173 to C197, C174 to C198, C247 to C199, C248 to C200, C184 to C201, C183 to C202, C182 to C203, C179 to C204, C178 to C205, C177 to C206, C249 to C207, C250 to C208, C251 to C209, C252 to C210, C253 to C211, C254 to C212, C199 to C213, C198 to C214, C197 to C215, C196 to C216, C195 to C217, C255 to C218, C256 to C219, C257 to C220, C258 to C221, C259 to C222, C328 to C223, C202 to C224, C201 to C225, C200 to C226, C260 to C227, C261 to C228, C262 to C229, C263 to C230, C331 to C231, C330 to C232, C181 to C233, C180 to C234, C264 to C235, C265 to C236, C266 to C237, C267 to C238, C211 to C239, C329 to C240, C268 to C241, C269 to C242, C213 to C243, C270 to C244, C175 to C245, C176 to C246, C185 to C247, C186 to C248, C187 to C249, C188 to C250, C189 to C251, C190 to C252, C191 to C253, C192 to C254, C193 to C255, C194 to C256, C203 to C257, C204 to C258, C205 to C259, C206 to C260, C207 to C261, C208 to C262, C209 to C263, C210 to C264, C212 to C265, C214 to C266, C215 to C267, C216 to C268, C217 to C269, C271 to C270, C272 to C271, C218 to C272, C332 to C281, C333 to C282, C334 to C283, C335 to C284, C336 to C285, C337 to C286, C338 to C287, C339 to C288, C340 to C289, C341 to C290, C342 to C291, C343 to C292, C344 to C293, C219 to C294, C220 to C295, C221 to C296, C222 to C297, C345 to C298, C346 to C299, C223 to C300, C224 to C301, C225 to C302, C226 to C303, C227 to C304, C228 to C305, C347 to C306, C229 to C307, C230 to C308, C231 to C309, C232 to C310, C233 to C311, C234 to C312, C235 to C313, C236 to C314, C237 to C315, C238 to C316, C239 to C317, C240 to C318, C241 to C319, C242 to C320, C243 to C321, C244 to C322, D2 to D28, D5 to D29, D3 to D30, D6 to D31, D4 to D32, J16 to J19, J18 to J20, J17 to J21, L3 to L2, L6 to L3, L7 to L5, L5 to L6, R213 to R117, R211 to R118, R212 to R119, R88 to R120, R89 to R121, R90 to R122, R52 to R123, R51 to R124, R123 to R125, R48 to R126, R46 to R127, R43 to R128, R91 to R129, R42 to R130, R92 to R131, R93 to R132, R94 to R133, R95 to R134, R96 to R135, R97 to R136, R41 to R137, R55 to R138, R56 to R139, R57 to R140, R98 to R141, R58 to R142, R99 to R143, R100 to R144, R101 to R145, R102 to R146, R63 to R147, R64 to R148, R103 to R149, R104 to R150, R44 to R151, R45 to R152, R47 to R153, R49 to R154, R50 to R155, R53 to R156, R54 to R157, R59 to R158, R60 to R159, R61 to R160, R62 to R161, R65 to R162, R105 to R163, R66 to R164, R124 to R165, R125 to R166, R67 to R167, R68 to R168, R69 to R169, R70 to R170, R126 to R171, R127 to R172, R214 to R173, R215 to R174, R216 to R175, R217 to R176, R218 to R177, R71 to R178, R72 to R179, R73 to R180, R219 to R181, R220 to R182, R221 to R183, R222 to R184, R223 to R185, R74 to R186, R224 to R187, R225 to R188, R75 to R189, R76 to R190, R77 to R191, R78 to R192, R79 to R193, R80 to R194, R81 to R195, R82 to R196, R83 to R197, R84 to R198, R85 to R199, R86 to R200, R87 to R201, TR4 to TR2, TR2 to TR3, TR5 to TR4, TR3 to TR5, U16 to U10, U18 to U11, U5 to U12, U6 to U13, U19 to U14, U20 to U15, U7 to U16, U8 to U17, U4 to U8, U17 to U9, Y1 to Y2, Y4 to Y3, Y2 to Y4, Y3 to Y6

Commit message: Add TVS diodes for ESD protection
Parts:
- added U23, U24, U25, U26, U27, U28, U29, U30, U31, U32: H5VU25U, Package_DFN_QFN:Diodes_UDFN-10_1.0x2.5mm_P0.5mm, symbol Power_Protection:D3V3XA4B10LP
- U10, U11, U13, U15, U17: value W25Q128JVS -> ZD25Q64BSIGT
Connections:
- net GND: now also U23.3 (VSS), U23.8 (VSS), U24.3 (VSS), U24.8 (VSS), U25.3 (VSS), U25.8 (VSS), U26.3 (VSS), U26.8 (VSS), U27.3 (VSS), U27.8 (VSS), U28.3 (VSS), U28.8 (VSS), U29.3 (VSS), U29.8 (VSS), U30.3 (VSS), U30.8 (VSS), U31.3 (VSS), U31.8 (VSS), U32.3 (VSS), U32.8 (VSS)
- net at R201.1: now also J20.22; no longer J21.22
- net at J20.20, TR4.13 (MX4-): now also U32.4
- net at J20.19, TR4.14 (MX4+): now also U32.5
- net at J20.17, TR4.16 (MX3-): now also U32.1
- net at J20.16, TR4.17 (MX3+): now also U31.4
- net at J20.18, TR4.19 (MX2-): now also U32.2
- net at J20.15, TR4.20 (MX2+): now also U31.5
- net at J20.14, TR4.22 (MX1-): now also U31.2
- net at J20.13, TR4.23 (MX1+): now also U31.1
- net at J20.8, TR2.13 (MX4-): now also U30.4
- net at J20.7, TR2.14 (MX4+): now also U30.5
- net at J20.5, TR2.16 (MX3-): now also U30.1
- net at J20.4, TR2.17 (MX3+): now also U29.4
- net at J20.6, TR2.19 (MX2-): now also U30.2
- net at J20.3, TR2.20 (MX2+): now also U29.5
- net at J20.2, TR2.22 (MX1-): now also U29.2
- net at J20.1, TR2.23 (MX1+): now also U29.1
- net at R170.1: now also J21.22; no longer J21.10
- net at R187.1: now also J20.12; no longer J20.24
- net at J20.10: now also R188.1; no longer R150.1
- net at J21.13, TR5.23 (MX1+): now also U27.1
- net at J21.14, TR5.22 (MX1-): now also U27.2
- net at J21.15, TR5.20 (MX2+): now also U27.5
- net at J21.16, TR5.17 (MX3+): now also U27.4
- net at J21.17, TR5.16 (MX3-): now also U28.1
- net at J21.18, TR5.19 (MX2-): now also U28.2
- net at J21.19, TR5.14 (MX4+): now also U28.5
- net at J21.20, TR5.13 (MX4-): now also U28.4
- net at J21.24: now also R169.1; no longer R200.1
- net at R149.1: now also J21.12; no longer J20.12
- net at J21.8, TR3.13 (MX4-): now also U26.4
- net at J21.7, TR3.14 (MX4+): now also U26.5
- net at J21.5, TR3.16 (MX3-): now also U26.1
- net at J21.4, TR3.17 (MX3+): now also U25.4
- net at J21.6, TR3.19 (MX2-): now also U26.2
- net at J21.3, TR3.20 (MX2+): now also U25.5
- net at J21.2, TR3.22 (MX1-): now also U25.2
- net at J21.1, TR3.23 (MX1+): now also U25.1
- net at J19.8, TR1.13 (MX4-): now also U24.4
- net at J19.7, TR1.14 (MX4+): now also U24.5
- net at J19.5, TR1.16 (MX3-): now also U24.1
- net at J19.4, TR1.17 (MX3+): now also U23.4
- net at J19.6, TR1.19 (MX2-): now also U24.2
- net at J19.3, TR1.20 (MX2+): now also U23.5
- net at J19.2, TR1.22 (MX1-): now also U23.2
- net at J19.1, TR1.23 (MX1+): now also U23.1
- new net: J20.24, R200.1
- new net: J21.10, R150.1
Other:
- moved on the sheet: C195, C196, C199, C200, C207, C208, C209, C210, C211, C212, C218, C219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

Commit message: Fix esd diodes, add some footprints.
Parts:
- removed C239, C298, C320: 390pF, symbol Device:C
- removed C293: 22uF, symbol Device:C_Small
- removed C294: 18pF, symbol Device:C_Small
- removed C321: 100nF, symbol Device:C_Small
- removed R201: 510R, symbol Device:R_Small
- removed U10, U17: ZD25Q64BSIGT, Package_SO:SOIC-8_5.3x5.3mm_P1.27mm, symbol Memory_Flash:W25Q128JVS
- removed U14, U16: KTI226V, Package_DFN_QFN:QFN-56-1EP_7x7mm_P0.4mm_EP5.6x5.6mm_ThermalVias, symbol custom:KTI226V
- removed U27, U28: H5VU25U, Package_DFN_QFN:Diodes_UDFN-10_1.0x2.5mm_P0.5mm, symbol Power_Protection:D3V3XA4B10LP
- added C239, C320: 100nF, symbol Device:C_Small
- added C293, C294, C321: 390pF, symbol Device:C
- added C298: 27pF, symbol Device:C_Small
- added R113: 10k, symbol Device:R_Small
- added U10, U27: KTI226V, Package_DFN_QFN:QFN-56-1EP_7x7mm_P0.4mm_EP5.6x5.6mm_ThermalVias, symbol custom:KTI226V
- added U14, U28: ZD25Q64BSIGT, Package_SO:SOIC-8_5.3x5.3mm_P1.27mm, symbol Memory_Flash:W25Q128JVS
- added U16, U17: H5VU25U, Package_DFN_QFN:Diodes_UDFN-10_1.0x2.5mm_P0.5mm, symbol Power_Protection:D3V3XA4B10LP
- C193, C194, C195, C196, C245, C246: value 18pF -> 27pF
- C197, C198, C297: value 220nF -> 27pF
- C201, C202, C203, C299, C300: value 100nF -> 220nF
- C204: value 22uF -> 220nF
- C205, C206, C233, C234, C278, C279, C280, C292, C303: value 22uF -> 100nF
- C214, C215, C216, C225, C226, C231, C285, C286, C289, C290: value 100nF -> 22uF
- C243: value 100pF -> 100nF
- C270, C271: value 18pF -> 100nF
- C273, C274: value 220nF -> 100nF
- C295: value 18pF -> 100pF
- C296: value 220nF -> 100pF
- C306: value 100pF -> 22uF
- J19: footprint (none) -> RJE361882145:AMPHENOL_RJE361882415
- R117, R123: value 10k -> 200R
- R118, R165: value 200R -> 10k
- R125, R190: value 22k -> 10k
- R130, R189: value 10k -> 22k
- R137, R147, R148: value 510R -> 10k
- R138: value 75R -> 22k
- R139, R140, R142, R182, R184, R185: value 75R -> 10k
- R166, R178, R180, R194: value 10k -> 510R
- R170, R195: value 510R -> 75R
- R171, R172, R174, R175, R176, R177: value 10k -> 75R
- R173: value 22k -> 75R
- R179: value 200R -> 510R
- R183: value 75R -> 200R
- R199: value 75R -> 510R
Connections:
- net +3V3: now also R137.2, R139.2, R140.2, R142.2, R147.2, R148.2, R163.2, R165.2, R186.2, R190.2; no longer R124.2, R126.2, R130.2, R172.2, R174.2, R175.2, R176.2, R177.2, R189.2, R194.2
- net +3V3SB: now also C213.2, C214.2, C215.2, C216.2, C217.2, C223.2, C224.2, C225.2, C226.2, C231.2, C232.1, C233.1, C234.1, C243.1, C270.1, C271.1, C273.1, C274.1, C291.1, C292.1, C306.2, R118.1, R124.1, R166.2, R178.2, R179.2, R180.2, R182.1, R184.1, R194.2, R199.2, C239.1, C320.1, R113.1, U10.14 (+3.3V_PAD), U10.23 (+3.3V_VPH), U10.33 (+3.3V_PAD), U10.39 (+3.3V_XO), U10.43 (+3.3V_CDB), U10.47 (+3.3V_A), U10.53 (+3.3V_A), U10.7 (+3.3V_DC), U14.8 (VCC), U27.14 (+3.3V_PAD), U27.23 (+3.3V_VPH), U27.33 (+3.3V_PAD), U27.39 (+3.3V_XO), U27.43 (+3.3V_CDB), U27.47 (+3.3V_A), U27.53 (+3.3V_A), U27.7 (+3.3V_DC), U28.8 (VCC); no longer C201.2, C202.2, C203.2, C204.2, C213.1, C214.1, C215.1, C216.1, C217.1, C275.2, C276.2, C277.2, C278.2, C279.2, C280.2, C281.1, C282.1, C283.1, C284.1, C285.1, C299.1, C300.2, R117.1, R137.2, R147.2, R148.2, R163.1, R166.1, R170.2, R178.1, R180.1, R195.2
- net ETH0.REFCLK+: now also U10.21 (PE_CLK_P); no longer U8.21 (PE_CLK_P)
- net ETH0.REFCLK-: now also U10.22 (PE_CLK_N); no longer U8.22 (PE_CLK_N)
- net ETH0.Rx0+: now also C203.1; no longer C197.1
- net ETH0.Rx0-: now also C204.1; no longer C198.1
- net ETH0.SMBCLK: now also U10.11 (SMB_CLK); no longer U8.11 (SMB_CLK)
- net ETH0.SMBDAT: now also U10.10 (SMB_DATA), U10.4 (ULP_WAKE_N); no longer U8.10 (SMB_DATA), U8.4 (ULP_WAKE_N)
- net ETH0.Tx0+: now also U10.28 (PE_Rx_P); no longer U8.28 (PE_Rx_P)
- net ETH0.Tx0-: now also U10.27 (PE_Rx_N); no longer U8.27 (PE_Rx_N)
- net ETH0.~{PLTRST}: now also U10.13 (PE_RST_N); no longer U8.13 (PE_RST_N)
- net ETH0.~{WAKE}: now also U10.12 (PE_WAKE_N); no longer U8.12 (PE_WAKE_N)
- net ETH2.REFCLK+: now also U8.21 (PE_CLK_P)
- net ETH2.REFCLK-: now also U8.22 (PE_CLK_N)
- net ETH2.Rx0+: now also C201.1; no longer C296.1
- net ETH2.Rx0-: now also C202.1; no longer C297.1
- net ETH2.SMBCLK: now also U8.11 (SMB_CLK)
- net ETH2.SMBDAT: now also U8.10 (SMB_DATA), U8.4 (ULP_WAKE_N)
- net ETH2.Tx0+: now also U8.28 (PE_Rx_P)
- net ETH2.Tx0-: now also U8.27 (PE_Rx_N)
- net ETH2.~{PLTRST}: now also U8.13 (PE_RST_N)
- net ETH2.~{WAKE}: now also U8.12 (PE_WAKE_N)
- net ETH4.REFCLK+: now also U27.21 (PE_CLK_P)
- net ETH4.REFCLK-: now also U27.22 (PE_CLK_N)
- net ETH4.Rx0+: now also C299.1; no longer C273.1
- net ETH4.Rx0-: now also C300.1; no longer C274.1
- net ETH4.SMBCLK: now also U27.11 (SMB_CLK)
- net ETH4.SMBDAT: now also U27.10 (SMB_DATA), U27.4 (ULP_WAKE_N)
- net ETH4.Tx0+: now also U27.28 (PE_Rx_P)
- net ETH4.Tx0-: now also U27.27 (PE_Rx_N)
- net ETH4.~{PLTRST}: now also U27.13 (PE_RST_N)
- net ETH4.~{WAKE}: now also U27.12 (PE_WAKE_N)
- net GND: now also C197.1, C198.1, C213.1, C214.1, C215.1, C216.1, C217.1, C231.1, C241.2, C270.2, C271.2, C273.2, C274.2, C281.1, C282.1, C286.2, C287.2, C288.2, C289.2, C295.2, C296.2, C297.1, C306.1, R117.1, R123.1, R126.2, R130.2, R138.2, R183.1, R185.2, R189.2, C239.2, C293.2, C294.1, C298.1, C320.2, C321.2, U10.57 (EPAD), U10.8 (Reserved), U14.4 (GND), U16.3 (VSS), U16.8 (VSS), U17.3 (VSS), U17.8 (VSS), U27.57 (EPAD), U27.8 (Reserved), U28.4 (GND); no longer C201.1, C202.1, C203.1, C204.1, C213.2, C214.2, C215.2, C216.2, C217.2, C231.2, C241.1, C270.1, C271.1, C281.2, C282.2, C286.1, C287.1, C288.1, C289.1, C295.1, C299.2, C300.1, C306.2, R118.1, R123.2, R165.1, R171.2, R173.2, R179.1, R186.2, R190.2
- net at R117.2: now also U8.20 (RBIAS); no longer U8.2 (LAN_DISABLE_N)
- net at R118.2: now also U10.2 (LAN_DISABLE_N); no longer U8.20 (RBIAS)
- net at U8.24 (PE_Tx_N): now also C202.2; no longer C198.2
- net at C197.2: now also Y5.1, U10.41 (XTAL_IN); no longer U8.25 (PE_Tx_P)
- net at U8.31 (LED1): now also J20.21; no longer J19.D2
- net at U8.32 (LED0): now also J20.23; no longer J19.D4
- net at R126.1: now also U15.6 (CLK), U10.35 (SPI_CLK); no longer U8.34 (SPI_DOUT/SEC_ENA)
- net at U8.35 (SPI_CLK): now also R125.1, U14.6 (CLK); no longer R123.1
- net at U8.36 (SPI_DIN/AUX_PWR): now also R127.1, U14.2 (DO/IO_{1}); no longer R124.1
- net at U8.37 (SPI_CS_N/PCIE_ENA): now also R140.1, U14.1 (~{CS}); no longer R127.1
- net at U8.42 (PHY_CAL): now also R130.1; no longer R125.1
- net at TR1.2 (TD1+), U8.45 (MDI_A_P): now also U23.4
- net at TR1.3 (TD1-), U8.46 (MDI_A_N): now also U23.5
- net at TR1.5 (TD2+), U8.48 (MDI_B_P): now also U23.2
- net at TR1.6 (TD2-), U8.49 (MDI_B_N): now also U23.1
- net at TR1.8 (TD3+), U8.51 (MDI_C_P): now also U16.4
- net at TR1.9 (TD3-), U8.52 (MDI_C_N): now also U16.5
- net at TR1.11 (TD4+), U8.54 (MDI_D_P): now also U16.2
- net at TR1.12 (TD4-), U8.55 (MDI_D_N): now also U16.1
- net at C312.2, C313.2, C314.2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: now also U27.26 (VDD_VP), U27.38 (VDD_CORE), U27.44 (VDD_A), U27.50 (VDD_A), U27.56 (VDD_A), U27.9 (VDD_CORE)
- net at TR4.1 (CT), TR4.10 (CT), TR4.4 (CT)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: now also C294.2
- net at TR4.11 (TD4+): now also U10.54 (MDI_D_P), U17.2
- net at TR4.12 (TD4-): now also U10.55 (MDI_D_N), U17.1
- net at TR4.15 (CT): now also R174.1; no longer R182.1
- net at TR4.18 (CT): now also R175.1; no longer R183.1
- net at TR4.2 (TD1+): now also U24.4, U10.45 (MDI_A_P)
- net at TR4.21 (CT): now also R176.1; no longer R184.1
- net at TR4.24 (CT): now also R177.1; no longer R185.1
- net at TR4.3 (TD1-): now also U24.5, U10.46 (MDI_A_N)
- net at TR4.5 (TD2+): now also U24.2, U10.48 (MDI_B_P)
- net at TR4.6 (TD2-): now also U24.1, U10.49 (MDI_B_N)
- net at TR4.8 (TD3+): now also U10.51 (MDI_C_P), U17.4
- net at TR4.9 (TD3-): now also U10.52 (MDI_C_N), U17.5
- net at TR2.1 (CT), TR2.10 (CT), TR2.4 (CT)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: now also C241.1; no longer C241.2
- net at TR2.11 (TD4+), U9.54 (MDI_D_P): now also U29.2
- net at TR2.12 (TD4-), U9.55 (MDI_D_N): now also U29.1
- net at TR2.2 (TD1+), U9.45 (MDI_A_P): now also U30.4
- net at TR2.3 (TD1-), U9.46 (MDI_A_N): now also U30.5
- net at TR2.5 (TD2+), U9.48 (MDI_B_P): now also U30.2
- net at TR2.6 (TD2-), U9.49 (MDI_B_N): now also U30.1
- net at TR2.8 (TD3+), U9.51 (MDI_C_P): now also U29.4
- net at TR2.9 (TD3-), U9.52 (MDI_C_N): now also U29.5
- net at J20.22: now also R179.1
- net at Y6.1: now also C297.2, U27.41 (XTAL_IN)
- net at J19.D1: now also R181.1; no longer R148.1
- net at U15.1 (~{CS}): now also R142.1, U10.37 (SPI_CS_N/PCIE_ENA); no longer R175.1
- net at R172.1: now also TR1.21 (CT); no longer U15.2 (DO/IO_{1})
- net at U15.3 (~{WP}/IO_{2}): now also R148.1; no longer R176.1
- net at U15.5 (DI/IO_{0}): now also R139.1, U10.34 (SPI_DOUT/SEC_ENA); no longer R174.1
- net at R171.1: now also TR1.18 (CT); no longer U15.6 (CLK)
- net at U15.7 (~{HOLD}/~{RESET}/IO_{3}): now also R165.1; no longer R177.1
- net at TR5.1 (CT), TR5.10 (CT), TR5.4 (CT)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: now also C321.1
- net at J21.24: now also R199.1; no longer R169.1
- net at Y5.3: now also C198.2, U10.40 (XTAL_OUT); no longer C271.2
- net at J21.21: now also U27.31 (LED1)
- net at R170.1: now also TR1.15 (CT); no longer J21.22
- net at J21.23: now also U27.32 (LED0)
- net at R137.1: now also U8.34 (SPI_DOUT/SEC_ENA), U14.5 (DI/IO_{0}); no longer D28.2 (A)
- net at U12.31 (LED1): now also J20.9; no longer J21.9
- net at U12.32 (LED0): now also J20.11; no longer J21.11
- net at TR3.2 (TD1+), U12.45 (MDI_A_P): now also U26.4
- net at TR3.3 (TD1-), U12.46 (MDI_A_N): now also U26.5
- net at TR3.5 (TD2+), U12.48 (MDI_B_P): now also U26.2
- net at TR3.6 (TD2-), U12.49 (MDI_B_N): now also U26.1
- net at TR3.8 (TD3+), U12.51 (MDI_C_P): now also U25.4
- net at TR3.9 (TD3-), U12.52 (MDI_C_N): now also U25.5
- net at TR3.11 (TD4+), U12.54 (MDI_D_P): now also U25.2
- net at TR3.12 (TD4-), U12.55 (MDI_D_N): now also U25.1
- net at R189.1: now also U27.42 (PHY_CAL)
- net at R191.1: now also U27.37 (SPI_CS_N/PCIE_ENA), U28.1 (~{CS})
- net at J20.10: now also R150.1; no longer R188.1
- net at U9.32 (LED0): now also J21.11; no longer J20.11
- net at J20.12: now also R149.1; no longer R187.1
- net at U9.31 (LED1): now also J21.9; no longer J20.9
- net at D31.2 (A): now also R169.1; no longer R181.1
- net at D32.1 (K): now also U27.30 (LED2)
- net at R186.1: now also U27.36 (SPI_DIN/AUX_PWR), U28.2 (DO/IO_{1})
- net at R192.1: now also U28.3 (~{WP}/IO_{2})
- net at Y6.3: now also C298.2, U27.40 (XTAL_OUT); no longer C295.2
- net at R190.1: now also U27.34 (SPI_DOUT/SEC_ENA), U28.5 (DI/IO_{0})
- net at TR5.2 (TD1+): now also U32.4, U27.45 (MDI_A_P)
- net at TR5.3 (TD1-): now also U32.5, U27.46 (MDI_A_N)
- net at TR5.5 (TD2+): now also U32.2, U27.48 (MDI_B_P)
- net at TR5.6 (TD2-): now also U32.1, U27.49 (MDI_B_N)
- net at L6.2: now also U27.5 (VDD_CTRL), U27.6 (VDD_CTRL)
- net at TR5.8 (TD3+): now also U31.4, U27.51 (MDI_C_P)
- net at TR5.9 (TD3-): now also U31.5, U27.52 (MDI_C_N)
- net at TR5.11 (TD4+): now also U31.2, U27.54 (MDI_D_P)
- net at TR5.12 (TD4-): now also U31.1, U27.55 (MDI_D_N)
- net at TR5.18 (CT): now also R196.1; no longer R197.1
- net at C322.1, R196.2, R197.2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: now also R195.2; no longer R199.2
- net at TR1.24 (CT): now also R173.1; no longer R142.1
- net at D31.1 (K): now also U10.30 (LED2)
- net at J19.D3: now also R180.1; no longer R147.1
- net at J20.24: now also R178.1; no longer R200.1
- net at R128.1: now also U15.2 (DO/IO_{1}), U10.36 (SPI_DIN/AUX_PWR)
- net at R195.1: now also TR5.15 (CT); no longer D32.2 (A)
- net at TR5.21 (CT): now also R197.1; no longer R198.1
- net at TR5.24 (CT): now also R198.1; no longer R199.1
- net at TR1.1 (CT), TR1.10 (CT), TR1.4 (CT)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: now also C293.1
- net at R193.1: now also U28.7 (~{HOLD}/~{RESET}/IO_{3})
- net at R194.1: now also D32.2 (A)
- net at R138.1: now also U10.42 (PHY_CAL); no longer TR1.15 (CT)
- net at L5.2: now also U10.5 (VDD_CTRL), U10.6 (VDD_CTRL)
- net at J21.12: now also R187.1; no longer R149.1
- net at J21.10: now also R188.1; no longer R150.1
- new net: C296.1, R174.2, R175.2, R176.2, R177.2
- new net: C275.2, C276.2, C277.2, C278.2, C283.1, C284.1, C285.1, C286.1, L2.1, U8.26 (VDD_VP), U8.38 (VDD_CORE), U8.44 (VDD_A), U8.50 (VDD_A), U8.56 (VDD_A), U8.9 (VDD_CORE)
- new net: C279.2, C280.2, C281.2, C282.2, C287.1, C288.1, C289.1, C290.1, L5.1, U10.26 (VDD_VP), U10.38 (VDD_CORE), U10.44 (VDD_A), U10.50 (VDD_A), U10.56 (VDD_A), U10.9 (VDD_CORE)
- new net: J21.8, TR2.13 (MX4-)
- new net: J21.7, TR2.14 (MX4+)
- new net: J21.5, TR2.16 (MX3-)
- new net: J21.4, TR2.17 (MX3+)
- new net: J21.6, TR2.19 (MX2-)
- new net: J21.3, TR2.20 (MX2+)
- new net: J21.2, TR2.22 (MX1-)
- new net: J21.1, TR2.23 (MX1+)
- new net: C295.1, R170.2, R171.2, R172.2, R173.2
- new net: R185.1, U27.35 (SPI_CLK), U28.6 (CLK)
- new net: J20.13, TR1.23 (MX1+)
- new net: J20.14, TR1.22 (MX1-)
- new net: J20.15, TR1.20 (MX2+)
- new net: J20.16, TR1.17 (MX3+)
- new net: J20.17, TR1.16 (MX3-)
- new net: J20.18, TR1.19 (MX2-)
- new net: J20.19, TR1.14 (MX4+)
- new net: J20.20, TR1.13 (MX4-)
- new net: R184.2, U27.1 (LAN_PWR_GOOD)
- new net: R182.2, U27.2 (LAN_DISABLE_N)
- new net: R183.2, U27.20 (RBIAS)
- new net: J20.1, TR3.23 (MX1+)
- new net: J20.2, TR3.22 (MX1-)
- new net: J20.3, TR3.20 (MX2+)
- new net: J20.4, TR3.17 (MX3+)
- new net: J20.5, TR3.16 (MX3-)
- new net: J20.6, TR3.19 (MX2-)
- new net: J20.7, TR3.14 (MX4+)
- new net: J20.8, TR3.13 (MX4-)
- new net: J21.22, R200.1
- new net: C203.2, U10.25 (PE_Tx_P)
- new net: R113.2, U8.2 (LAN_DISABLE_N)
- new net: C299.2, U27.25 (PE_Tx_P)
- new net: C300.2, U27.24 (PE_Tx_N)
- new net: J19.8, TR4.13 (MX4-)
- new net: J19.7, TR4.14 (MX4+)
- new net: J19.5, TR4.16 (MX3-)
- new net: J19.4, TR4.17 (MX3+)
- new net: J19.6, TR4.19 (MX2-)
- new net: J19.3, TR4.20 (MX2+)
- new net: J19.2, TR4.22 (MX1-)
- new net: J19.1, TR4.23 (MX1+)
- new net: D28.2 (A), R166.1
- new net: C201.2, U8.25 (PE_Tx_P)
- new net: R147.1, U14.3 (~{WP}/IO_{2})
- new net: R163.1, U14.7 (~{HOLD}/~{RESET}/IO_{3})
- new net: J19.D2, U10.31 (LED1)
- new net: J19.D4, U10.32 (LED0)
- new net: R123.2, U10.20 (RBIAS)
- new net: C204.2, U10.24 (PE_Tx_N)
- new net: R124.2, U10.1 (LAN_PWR_GOOD)
Other:
- moved on the sheet: C241, C244, C268, C272, R143, R144, R145, R146, R149, R150, R162, R164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

Commit message: Add more footprints
Parts:
- Y2, Y3, Y4, Y5, Y6: footprint (none) -> Crystal:Crystal_SMD_3225-4Pin_3.2x2.5mm
Changed lines of the file:
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@@
 			)
 		)
-		(property "Footprint" ""
+		(property "Footprint" "Crystal:Crystal_SMD_3225-4Pin_3.2x2.5mm"
 			(at 35.56 378.46 0)
 			(effects
@@
 			)
 		)
-		(property "Footprint" ""
+		(property "Footprint" "Crystal:Crystal_SMD_3225-4Pin_3.2x2.5mm"
 			(at 39.37 241.3 0)
 			(effects
@@
 			)
 		)
-		(property "Footprint" ""
+		(property "Footprint" "Crystal:Crystal_SMD_3225-4Pin_3.2x2.5mm"
 			(at 41.91 123.19 0)
 			(effects
@@
 			)
 		)
-		(property "Footprint" ""
+		(property "Footprint" "Crystal:Crystal_SMD_3225-4Pin_3.2x2.5mm"
 			(at 313.69 243.84 0)
 			(effects
@@
 			)
 		)
-		(property "Footprint" ""
+		(property "Footprint" "Crystal:Crystal_SMD_3225-4Pin_3.2x2.5mm"
 			(at 316.23 125.73 0)
 			(effects

Commit message: Add USB Type E Header Footprint
Parts:
- J19: symbol custom:1xRJ45+2xUSB3 -> Custom:1xRJ45+2xUSB3
- U10, U12, U27, U8, U9: symbol custom:KTI226V -> Custom:KTI226V
Changed lines of the file:
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@@
 	)
 	(symbol
-		(lib_id "custom:KTI226V")
+		(lib_id "Custom:KTI226V")
 		(at 359.41 50.8 0)
 		(unit 1)
@@
 	)
 	(symbol
-		(lib_id "custom:KTI226V")
+		(lib_id "Custom:KTI226V")
 		(at 356.87 168.91 0)
 		(unit 1)
@@
 	)
 	(symbol
-		(lib_id "custom:KTI226V")
+		(lib_id "Custom:KTI226V")
 		(at 82.55 166.37 0)
 		(unit 1)
@@
 	)
 	(symbol
-		(lib_id "custom:1xRJ45+2xUSB3")
+		(lib_id "Custom:1xRJ45+2xUSB3")
 		(at 236.22 90.17 180)
 		(unit 1)
@@
 	)
 	(symbol
-		(lib_id "custom:KTI226V")
+		(lib_id "Custom:KTI226V")
 		(at 78.74 303.53 0)
 		(unit 1)
@@
 	)
 	(symbol
-		(lib_id "custom:KTI226V")
+		(lib_id "Custom:KTI226V")
 		(at 85.09 48.26 0)
 		(unit 1)
