File: KiCad/eth.kicad_sch (KiCad schematic)
At the start: 258 parts, among them J19 RJ45_LED_Shielded_x2, J20 RJE361882415, J21 RJ45_LED_Shielded_x2, U10 H5VU25U, U11 H5VU25U, U12 KTI226V, U13 KTI226V, U14 ZD25Q64BSIGT, U15 ZD25Q64BSIGT, U16 H5VU25U, U17 H5VU25U, U18 H5VU25U, U19 H5VU25U, U20 KTI226V, U21 KTI226V, U22 ZD25Q64BSIGT, U23 ZD25Q64BSIGT, U24 H5VU25U, U25 H5VU25U, U26 KTI226V, U27 ZD25Q64BSIGT, U8 H5VU25U, U9 H5VU25U, Y2 25MHz, Y3 25MHz, Y4 25MHz, Y5 25MHz, Y6 25MHz

Commit message: Arranging components
Connections:
- net at U16.1, U20.55 (MDI_D_N): now also TR3.2 (TD1+); no longer TR3.12 (TD4-)
- net at U16.2, U20.54 (MDI_D_P): now also TR3.3 (TD1-); no longer TR3.11 (TD4+)
- net at U16.4, U20.51 (MDI_C_P): now also TR3.6 (TD2-); no longer TR3.8 (TD3+)
- net at U16.5, U20.52 (MDI_C_N): now also TR3.5 (TD2+); no longer TR3.9 (TD3-)
- net at R131.1: now also TR1.15 (CT); no longer TR1.24 (CT)
- net at U12.55 (MDI_D_N), U8.1: now also TR1.2 (TD1+); no longer TR1.12 (TD4-)
- net at U12.54 (MDI_D_P), U8.2: now also TR1.3 (TD1-); no longer TR1.11 (TD4+)
- net at U12.51 (MDI_C_P), U8.4: now also TR1.6 (TD2-); no longer TR1.8 (TD3+)
- net at U12.52 (MDI_C_N), U8.5: now also TR1.5 (TD2+); no longer TR1.9 (TD3-)
- net at R191.1: now also TR5.21 (CT); no longer TR5.18 (CT)
- net at U18.1, U21.55 (MDI_D_N): now also TR4.2 (TD1+); no longer TR4.12 (TD4-)
- net at U18.2, U21.54 (MDI_D_P): now also TR4.3 (TD1-); no longer TR4.11 (TD4+)
- net at U18.4, U21.51 (MDI_C_P): now also TR4.6 (TD2-); no longer TR4.8 (TD3+)
- net at U18.5, U21.52 (MDI_C_N): now also TR4.5 (TD2+); no longer TR4.9 (TD3-)
- net at TR4.13 (MX4-): now also J21.1; no longer J21.8
- net at TR4.14 (MX4+): now also J21.2; no longer J21.7
- net at TR4.15 (CT): now also R169.1; no longer R166.1
- net at TR4.16 (MX3-): now also J21.3; no longer J21.5
- net at TR4.17 (MX3+): now also J21.6; no longer J21.4
- net at TR4.18 (CT): now also R168.1; no longer R167.1
- net at TR4.19 (MX2-): now also J21.4; no longer J21.6
- net at U19.4, U21.45 (MDI_A_P): now also TR4.12 (TD4-); no longer TR4.2 (TD1+)
- net at TR4.20 (MX2+): now also J21.5; no longer J21.3
- net at TR4.21 (CT): now also R167.1; no longer R168.1
- net at TR4.22 (MX1-): now also J21.7; no longer J21.2
- net at TR4.23 (MX1+): now also J21.8; no longer J21.1
- net at TR4.24 (CT): now also R166.1; no longer R169.1
- net at U19.5, U21.46 (MDI_A_N): now also TR4.11 (TD4+); no longer TR4.3 (TD1-)
- net at U19.2, U21.48 (MDI_B_P): now also TR4.9 (TD3-); no longer TR4.5 (TD2+)
- net at U19.1, U21.49 (MDI_B_N): now also TR4.8 (TD3+); no longer TR4.6 (TD2-)
- net at R163.1: now also TR3.21 (CT); no longer TR3.18 (CT)
- net at R192.1: now also TR5.18 (CT); no longer TR5.21 (CT)
- net at R130.1: now also TR1.18 (CT); no longer TR1.21 (CT)
- net at R162.1: now also TR3.24 (CT); no longer TR3.15 (CT)
- net at R135.1: now also TR2.15 (CT); no longer TR2.24 (CT)
- net at R129.1: now also TR1.21 (CT); no longer TR1.18 (CT)
- net at U25.1, U26.49 (MDI_B_N): now also TR5.8 (TD3+); no longer TR5.6 (TD2-)
- net at U25.2, U26.48 (MDI_B_P): now also TR5.9 (TD3-); no longer TR5.5 (TD2+)
- net at U25.4, U26.45 (MDI_A_P): now also TR5.12 (TD4-); no longer TR5.2 (TD1+)
- net at U25.5, U26.46 (MDI_A_N): now also TR5.11 (TD4+); no longer TR5.3 (TD1-)
- net at J19.13: now also TR3.13 (MX4-); no longer TR3.23 (MX1+)
- net at J19.14: now also TR3.14 (MX4+); no longer TR3.22 (MX1-)
- net at J19.15: now also TR3.16 (MX3-); no longer TR3.20 (MX2+)
- net at J19.16: now also TR3.19 (MX2-); no longer TR3.17 (MX3+)
- net at J19.17: now also TR3.20 (MX2+); no longer TR3.16 (MX3-)
- net at J19.18: now also TR3.17 (MX3+); no longer TR3.19 (MX2-)
- net at J19.19: now also TR3.22 (MX1-); no longer TR3.14 (MX4+)
- net at J19.20: now also TR3.23 (MX1+); no longer TR3.13 (MX4-)
- net at U24.2, U26.54 (MDI_D_P): now also TR5.3 (TD1-); no longer TR5.11 (TD4+)
- net at U24.1, U26.55 (MDI_D_N): now also TR5.2 (TD1+); no longer TR5.12 (TD4-)
- net at TR5.13 (MX4-): now also J21.13; no longer J21.20
- net at TR5.14 (MX4+): now also J21.14; no longer J21.19
- net at TR5.15 (CT): now also R193.1; no longer R190.1
- net at TR5.16 (MX3-): now also J21.15; no longer J21.17
- net at TR5.17 (MX3+): now also J21.18; no longer J21.16
- net at TR5.19 (MX2-): now also J21.16; no longer J21.18
- net at TR5.20 (MX2+): now also J21.17; no longer J21.15
- net at TR5.22 (MX1-): now also J21.19; no longer J21.14
- net at TR5.23 (MX1+): now also J21.20; no longer J21.13
- net at TR5.24 (CT): now also R190.1; no longer R193.1
- net at U24.4, U26.51 (MDI_C_P): now also TR5.6 (TD2-); no longer TR5.8 (TD3+)
- net at U24.5, U26.52 (MDI_C_N): now also TR5.5 (TD2+); no longer TR5.9 (TD3-)
- net at R128.1: now also TR1.24 (CT); no longer TR1.15 (CT)
- net at U11.4, U13.45 (MDI_A_P): now also TR2.12 (TD4-); no longer TR2.2 (TD1+)
- net at U11.5, U13.46 (MDI_A_N): now also TR2.11 (TD4+); no longer TR2.3 (TD1-)
- net at U11.2, U13.48 (MDI_B_P): now also TR2.9 (TD3-); no longer TR2.5 (TD2+)
- net at U11.1, U13.49 (MDI_B_N): now also TR2.8 (TD3+); no longer TR2.6 (TD2-)
- net at U10.4, U13.51 (MDI_C_P): now also TR2.6 (TD2-); no longer TR2.8 (TD3+)
- net at U10.5, U13.52 (MDI_C_N): now also TR2.5 (TD2+); no longer TR2.9 (TD3-)
- net at U10.2, U13.54 (MDI_D_P): now also TR2.3 (TD1-); no longer TR2.11 (TD4+)
- net at U10.1, U13.55 (MDI_D_N): now also TR2.2 (TD1+); no longer TR2.12 (TD4-)
- net at J19.1: now also TR2.13 (MX4-); no longer TR2.23 (MX1+)
- net at J19.2: now also TR2.14 (MX4+); no longer TR2.22 (MX1-)
- net at J19.3: now also TR2.16 (MX3-); no longer TR2.20 (MX2+)
- net at J19.4: now also TR2.19 (MX2-); no longer TR2.17 (MX3+)
- net at J19.5: now also TR2.20 (MX2+); no longer TR2.16 (MX3-)
- net at J19.6: now also TR2.17 (MX3+); no longer TR2.19 (MX2-)
- net at J19.7: now also TR2.22 (MX1-); no longer TR2.14 (MX4+)
- net at J19.8: now also TR2.23 (MX1+); no longer TR2.13 (MX4-)
- net at R132.1: now also TR2.24 (CT); no longer TR2.15 (CT)
- net at TR2.18 (CT): now also R134.1; no longer R133.1
- net at TR2.21 (CT): now also R133.1; no longer R134.1
- net at TR1.13 (MX4-): now also J20.1; no longer J20.8
- net at TR1.14 (MX4+): now also J20.2; no longer J20.7
- net at TR1.16 (MX3-): now also J20.3; no longer J20.5
- net at TR1.17 (MX3+): now also J20.6; no longer J20.4
- net at TR1.19 (MX2-): now also J20.4; no longer J20.6
- net at U12.45 (MDI_A_P), U9.4: now also TR1.12 (TD4-); no longer TR1.2 (TD1+)
- net at TR1.20 (MX2+): now also J20.5; no longer J20.3
- net at TR1.22 (MX1-): now also J20.7; no longer J20.2
- net at TR1.23 (MX1+): now also J20.8; no longer J20.1
- net at U12.46 (MDI_A_N), U9.5: now also TR1.11 (TD4+); no longer TR1.3 (TD1-)
- net at U12.48 (MDI_B_P), U9.2: now also TR1.9 (TD3-); no longer TR1.5 (TD2+)
- net at U12.49 (MDI_B_N), U9.1: now also TR1.8 (TD3+); no longer TR1.6 (TD2-)
- net at U17.4, U20.45 (MDI_A_P): now also TR3.12 (TD4-); no longer TR3.2 (TD1+)
- net at U17.5, U20.46 (MDI_A_N): now also TR3.11 (TD4+); no longer TR3.3 (TD1-)
- net at U17.2, U20.48 (MDI_B_P): now also TR3.9 (TD3-); no longer TR3.5 (TD2+)
- net at U17.1, U20.49 (MDI_B_N): now also TR3.8 (TD3+); no longer TR3.6 (TD2-)
- net at R164.1: now also TR3.18 (CT); no longer TR3.21 (CT)
- net at R165.1: now also TR3.15 (CT); no longer TR3.24 (CT)
Changed lines of the file:
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@@
 		(lib_id "Transformer:30F-51NL")
 		(at 472.44 196.85 0)
+		(mirror x)
 		(unit 1)
 		(exclude_from_sim no)
@@
 		(dnp no)
 		(property "Reference" "TR4"
-			(at 472.44 171.45 0)
+			(at 472.44 175.006 0)
 			(effects
 				(font
@@
 		)
 		(property "Value" "QG2439S"
-			(at 472.44 173.99 0)
+			(at 472.44 172.466 0)
 			(effects
 				(font
@@
 		)
 		(property "Footprint" "Custom:QG2439S"
-			(at 464.82 189.23 0)
+			(at 464.82 204.47 0)
 			(effects
 				(font
@@
 		)
 		(property "Datasheet" "https://datasheet.lcsc.com/lcsc/1811051610_Shanghai-YDS-Tech-30F-51NL_C123168.pdf"
-			(at 472.44 219.71 0)
+			(at 472.44 173.99 0)
 			(effects
 				(font
@@
 		(lib_id "Transformer:30F-51NL")
 		(at 194.31 331.47 0)
+		(mirror x)
 		(unit 1)
 		(exclude_from_sim no)
@@
 		(dnp no)
 		(property "Reference" "TR5"
-			(at 194.31 306.07 0)
+			(at 194.31 309.626 0)
 			(effects
 				(font
@@
 		)
 		(property "Value" "QG2439S"
-			(at 194.31 308.61 0)
+			(at 194.31 307.086 0)
 			(effects
 				(font
@@
 		)
 		(property "Footprint" "Custom:QG2439S"
-			(at 186.69 323.85 0)
+			(at 186.69 339.09 0)
 			(effects
 				(font
@@
 		)
 		(property "Datasheet" "https://datasheet.lcsc.com/lcsc/1811051610_Shanghai-YDS-Tech-30F-51NL_C123168.pdf"
-			(at 194.31 354.33 0)
+			(at 194.31 308.61 0)
 			(effects
 				(font
@@
 		(lib_id "Transformer:30F-51NL")
 		(at 474.98 78.74 0)
+		(mirror x)
 		(unit 1)
 		(exclude_from_sim no)
@@
 		(on_board yes)
 		(dnp no)
-		(fields_autoplaced yes)
 		(property "Reference" "TR2"
-			(at 474.98 53.34 0)
+			(at 474.98 57.15 0)
 			(effects
 				(font
@@
 		)
 		(property "Value" "QG2439S"
-			(at 474.98 55.88 0)
+			(at 474.98 54.61 0)
 			(effects
 				(font
@@
 		)
 		(property "Footprint" "Custom:QG2439S"
-			(at 467.36 71.12 0)
+			(at 467.36 86.36 0)
 			(effects
 				(font
@@
 		)
 		(property "Datasheet" "https://datasheet.lcsc.com/lcsc/1811051610_Shanghai-YDS-Tech-30F-51NL_C123168.pdf"
-			(at 474.98 101.6 0)
+			(at 474.98 55.88 0)
 			(effects
 				(font
@@
 		(lib_id "Transformer:30F-51NL")
 		(at 200.66 76.2 0)
+		(mirror x)
 		(unit 1)
 		(exclude_from_sim no)
@@
 		(on_board yes)
 		(dnp no)
-		(fields_autoplaced yes)
 		(property "Reference" "TR1"
-			(at 200.66 50.8 0)
+			(at 200.66 54.61 0)
 			(effects
 				(font
@@
 		)
 		(property "Value" "QG2439S"
-			(at 200.66 53.34 0)
+			(at 200.66 52.324 0)
 			(effects
 				(font
@@
 		)
 		(property "Footprint" "Custom:QG2439S"
-			(at 193.04 68.58 0)
+			(at 193.04 83.82 0)
 			(effects
 				(font
@@
 		)
 		(property "Datasheet" "https://datasheet.lcsc.com/lcsc/1811051610_Shanghai-YDS-Tech-30F-51NL_C123168.pdf"
-			(at 200.66 99.06 0)
+			(at 200.66 53.34 0)
 			(effects
 				(font
@@
 		(lib_id "Transformer:30F-51NL")
 		(at 198.12 194.31 0)
+		(mirror x)
 		(unit 1)
 		(exclude_from_sim no)
@@
 		(dnp no)
 		(property "Reference" "TR3"
-			(at 198.12 168.91 0)
+			(at 198.12 172.212 0)
 			(effects
 				(font
@@
 		)
 		(property "Value" "QG2439S"
-			(at 198.12 171.45 0)
+			(at 198.12 169.672 0)
 			(effects
 				(font
@@
 		)
 		(property "Footprint" "Custom:QG2439S"
-			(at 190.5 186.69 0)
+			(at 190.5 201.93 0)
 			(effects
 				(font
@@
 		)
 		(property "Datasheet" "https://datasheet.lcsc.com/lcsc/1811051610_Shanghai-YDS-Tech-30F-51NL_C123168.pdf"
-			(at 198.12 217.17 0)
+			(at 198.12 171.45 0)
 			(effects
 				(font

Commit message: Re-annotate schematic
Parts:
- renumbered C193 to C203, C194 to C204, C195 to C205, C196 to C206, C197 to C207, C198 to C208, C199 to C209, C200 to C210, C201 to C211, C202 to C212, C203 to C213, C204 to C214, C205 to C215, C206 to C216, C207 to C217, C208 to C218, C209 to C219, C210 to C220, C211 to C221, C212 to C222, C213 to C223, C214 to C224, C215 to C225, C216 to C226, C217 to C227, C218 to C228, C219 to C229, C220 to C230, C221 to C231, C222 to C232, C223 to C233, C224 to C234, C225 to C235, C226 to C236, C227 to C237, C228 to C238, C229 to C239, C230 to C240, C231 to C241, C232 to C242, C233 to C243, C234 to C244, C235 to C245, C236 to C246, C237 to C247, C238 to C248, C239 to C249, C240 to C250, C241 to C251, C242 to C252, C243 to C253, C244 to C254, C245 to C255, C246 to C256, C247 to C257, C248 to C258, C249 to C259, C250 to C260, C251 to C261, C252 to C262, C253 to C263, C254 to C264, C255 to C265, C256 to C266, C257 to C267, C258 to C268, C259 to C269, C260 to C270, C261 to C271, C262 to C272, C263 to C273, C264 to C274, C265 to C275, C266 to C276, C267 to C277, C268 to C278, C269 to C279, C270 to C280, C271 to C281, C272 to C282, C273 to C283, C274 to C284, C275 to C285, C276 to C286, C277 to C287, C278 to C288, C279 to C289, C280 to C290, C281 to C291, C282 to C292, C283 to C293, C284 to C294, C285 to C295, C286 to C296, C287 to C297, C288 to C298, C289 to C299, C290 to C300, C291 to C301, C292 to C302, C293 to C303, C294 to C304, C295 to C305, C296 to C306, C297 to C307, C298 to C308, C299 to C309, C300 to C310, C301 to C311, C302 to C312, C303 to C313, C304 to C314, C305 to C315, C306 to C316, C307 to C317, C308 to C318, C309 to C319, C310 to C320, C311 to C321, C312 to C322, C313 to C323, C314 to C324, C315 to C325, C316 to C326, C317 to C327, C318 to C328, C319 to C329, C320 to C330, C321 to C331, C322 to C332, J19 to J18, J20 to J19, J21 to J20, R116 to R109, R117 to R110, R118 to R111, R119 to R112, R120 to R113, R121 to R114, R122 to R115, R123 to R116, R124 to R117, R125 to R118, R126 to R119, R127 to R120, R128 to R121, R129 to R122, R130 to R123, R131 to R124, R132 to R125, R133 to R126, R134 to R127, R135 to R128, R136 to R129, R137 to R130, R138 to R131, R139 to R132, R140 to R133, R141 to R134, R142 to R135, R143 to R136, R144 to R137, R145 to R138, R146 to R139, R147 to R140, R148 to R141, R149 to R142, R150 to R143, R151 to R144, R152 to R145, R153 to R146, R154 to R147, R155 to R148, R156 to R149, R157 to R150, R158 to R151, R159 to R152, R160 to R153, R161 to R154, R162 to R155, R163 to R156, R164 to R157, R165 to R158, R166 to R159, R167 to R160, R168 to R161, R169 to R162, R170 to R163, R171 to R164, R172 to R165, R173 to R166, R174 to R167, R175 to R168, R176 to R169, R177 to R170, R178 to R171, R179 to R172, R180 to R173, R181 to R174, R182 to R175, R183 to R176, R184 to R177, R185 to R178, R186 to R179, R187 to R180, R188 to R181, R189 to R182, R190 to R183, R191 to R184, R192 to R185, R193 to R186, R194 to R187, R195 to R188, R196 to R189, R197 to R190, R198 to R191, R199 to R192, R200 to R193
