File: KiCad/pcie.kicad_sch (KiCad schematic)
At the start: 32 parts, among them J6 Bus_PCI_Express_x4, J7 Bus_M.2_Socket_E, J8 Bus_M.2_Socket_E, J9 Bus_PCI_Express_x4

Commit message: Remove 0.95V Power Supply, Replace 3.3V Standby Power Supply
Connections:
- net SLOT2_M2E_PCIE.Rx0+ renamed SLOT2_M2E.Rx0+
- net SLOT2_M2E_PCIE.Rx0- renamed SLOT2_M2E.Rx0-
- net SLOT2_M2E_PCIE.Tx0+ renamed SLOT2_M2E.Tx0+
- net SLOT2_M2E_PCIE.Tx0- renamed SLOT2_M2E.Tx0-
- net SLOT3_M2E_PCIE.Rx0+ renamed SLOT3_M2E.Rx0+
- net SLOT3_M2E_PCIE.Rx0- renamed SLOT3_M2E.Rx0-
- net SLOT3_M2E_PCIE.Tx0+ renamed SLOT3_M2E.Tx0+
- net SLOT3_M2E_PCIE.Tx0- renamed SLOT3_M2E.Tx0-
- net SLOT4_PCIEx4.REFCLK+ renamed SLOT4x4.REFCLK+
- net SLOT4_PCIEx4.REFCLK- renamed SLOT4x4.REFCLK-
- net SLOT4_PCIEx4.Rx0+ renamed SLOT4x4.Rx0+
- net SLOT4_PCIEx4.Rx0- renamed SLOT4x4.Rx0-
- net SLOT4_PCIEx4.Rx1+ renamed SLOT4x4.Rx1+
- net SLOT4_PCIEx4.Rx1- renamed SLOT4x4.Rx1-
- net SLOT4_PCIEx4.Rx2+ renamed SLOT4x4.Rx2+
- net SLOT4_PCIEx4.Rx2- renamed SLOT4x4.Rx2-
- net SLOT4_PCIEx4.Rx3+ renamed SLOT4x4.Rx3+
- net SLOT4_PCIEx4.Rx3- renamed SLOT4x4.Rx3-
- net SLOT4_PCIEx4.SMBCLK renamed SLOT4x4.SMBCLK
- net SLOT4_PCIEx4.SMBDAT renamed SLOT4x4.SMBDAT
- net SLOT4_PCIEx4.Tx0+ renamed SLOT4x4.Tx0+
- net SLOT4_PCIEx4.Tx0- renamed SLOT4x4.Tx0-
- net SLOT4_PCIEx4.Tx1+ renamed SLOT4x4.Tx1+
- net SLOT4_PCIEx4.Tx1- renamed SLOT4x4.Tx1-
- net SLOT4_PCIEx4.Tx2+ renamed SLOT4x4.Tx2+
- net SLOT4_PCIEx4.Tx2- renamed SLOT4x4.Tx2-
- net SLOT4_PCIEx4.Tx3+ renamed SLOT4x4.Tx3+
- net SLOT4_PCIEx4.Tx3- renamed SLOT4x4.Tx3-
- net SLOT4_PCIEx4.~{PLTRST} renamed SLOT4x4.~{PLTRST}
- net SLOT4_PCIEx4.~{WAKE} renamed SLOT4x4.~{WAKE}
- net SLOT5_PCIEx4.REFCLK+ renamed SLOT5x4.REFCLK+
- net SLOT5_PCIEx4.REFCLK- renamed SLOT5x4.REFCLK-
- net SLOT5_PCIEx4.Rx0+ renamed SLOT5x4.Rx0+
- net SLOT5_PCIEx4.Rx0- renamed SLOT5x4.Rx0-
- net SLOT5_PCIEx4.Rx1+ renamed SLOT5x4.Rx1+
- net SLOT5_PCIEx4.Rx1- renamed SLOT5x4.Rx1-
- net SLOT5_PCIEx4.Rx2+ renamed SLOT5x4.Rx2+
- net SLOT5_PCIEx4.Rx2- renamed SLOT5x4.Rx2-
- net SLOT5_PCIEx4.Rx3+ renamed SLOT5x4.Rx3+
- net SLOT5_PCIEx4.Rx3- renamed SLOT5x4.Rx3-
- net SLOT5_PCIEx4.SMBCLK renamed SLOT5x4.SMBCLK
- net SLOT5_PCIEx4.SMBDAT renamed SLOT5x4.SMBDAT
- net SLOT5_PCIEx4.Tx0+ renamed SLOT5x4.Tx0+
- net SLOT5_PCIEx4.Tx0- renamed SLOT5x4.Tx0-
- net SLOT5_PCIEx4.Tx1+ renamed SLOT5x4.Tx1+
- net SLOT5_PCIEx4.Tx1- renamed SLOT5x4.Tx1-
- net SLOT5_PCIEx4.Tx2+ renamed SLOT5x4.Tx2+
- net SLOT5_PCIEx4.Tx2- renamed SLOT5x4.Tx2-
- net SLOT5_PCIEx4.Tx3+ renamed SLOT5x4.Tx3+
- net SLOT5_PCIEx4.Tx3- renamed SLOT5x4.Tx3-
- net SLOT5_PCIEx4.~{PLTRST} renamed SLOT5x4.~{PLTRST}
- net SLOT5_PCIEx4.~{WAKE} renamed SLOT5x4.~{WAKE}
- no-connect marks 92 -> 94

Commit message: Re-annotate components
Parts:
- renumbered C127 to C139, C128 to C140, C129 to C141, C130 to C142, C131 to C143, C132 to C144, C133 to C145, C134 to C146, C135 to C147, C136 to C148, C137 to C149, C138 to C150, C139 to C151, C140 to C152, C141 to C153, C142 to C154, C143 to C155, C144 to C156, C145 to C157, C146 to C158, C147 to C159, C148 to C160, C149 to C161, C150 to C162, R37 to R104, R38 to R105, R39 to R106, R40 to R107

Commit message: Add more footprints
Parts:
- C139, C140, C143, C144, C149, C151, C152, C155, C160, C161: footprint A_HDJ_Library:C_0402_1005Metric -> Capacitor_SMD:C_0603_1608Metric
- C141, C142, C150, C153, C154, C162: footprint A_HDJ_Library:CP_Elec_6.3x7.7 -> Capacitor_SMD:CP_Elec_6.3x7.7
- C145, C146, C147, C148, C156, C157, C158, C159: footprint (none) -> Capacitor_SMD:C_0603_1608Metric
Changed lines of the file:
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@@
 			)
 		)
-		(property "Footprint" "A_HDJ_Library:C_0402_1005Metric"
+		(property "Footprint" "Capacitor_SMD:C_0603_1608Metric"
 			(at 446.7352 241.3 0)
 			(effects
@@
 			)
 		)
-		(property "Footprint" "A_HDJ_Library:C_0402_1005Metric"
+		(property "Footprint" "Capacitor_SMD:C_0603_1608Metric"
 			(at 155.9052 256.54 0)
 			(effects
@@
 			)
 		)
-		(property "Footprint" "A_HDJ_Library:C_0402_1005Metric"
+		(property "Footprint" "Capacitor_SMD:C_0603_1608Metric"
 			(at 460.7052 262.89 0)
 			(effects
@@
 			)
 		)
-		(property "Footprint" "A_HDJ_Library:C_0402_1005Metric"
+		(property "Footprint" "Capacitor_SMD:C_0603_1608Metric"
 			(at 420.0652 262.89 0)
 			(effects
@@
 			)
 		)
-		(property "Footprint" "A_HDJ_Library:C_0402_1005Metric"
+		(property "Footprint" "Capacitor_SMD:C_0603_1608Metric"
 			(at 441.6552 241.3 0)
 			(effects
@@
 			)
 		)
-		(property "Footprint" ""
+		(property "Footprint" "Capacitor_SMD:C_0603_1608Metric"
 			(at 147.32 63.5 0)
 			(effects
@@
 			)
 		)
-		(property "Footprint" "A_HDJ_Library:CP_Elec_6.3x7.7"
+		(property "Footprint" "Capacitor_SMD:CP_Elec_6.3x7.7"
 			(at 160.9852 256.54 0)
 			(effects
@@
 			)
 		)
-		(property "Footprint" ""
+		(property "Footprint" "Capacitor_SMD:C_0603_1608Metric"
 			(at 147.32 74.93 0)
 			(effects
@@
 			)
 		)
-		(property "Footprint" ""
+		(property "Footprint" "Capacitor_SMD:C_0603_1608Metric"
 			(at 443.23 77.47 0)
 			(effects
@@
 			)
 		)
-		(property "Footprint" ""
+		(property "Footprint" "Capacitor_SMD:C_0603_1608Metric"
 			(at 443.23 69.85 0)
 			(effects
@@
 			)
 		)
-		(property "Footprint" "A_HDJ_Library:C_0402_1005Metric"
+		(property "Footprint" "Capacitor_SMD:C_0603_1608Metric"
 			(at 115.2652 256.54 0)
 			(effects
@@
 			)
 		)
-		(property "Footprint" "A_HDJ_Library:CP_Elec_6.3x7.7"
+		(property "Footprint" "Capacitor_SMD:CP_Elec_6.3x7.7"
 			(at 430.2252 262.89 0)
 			(effects
@@
 			)
 		)
-		(property "Footprint" "A_HDJ_Library:C_0402_1005Metric"
+		(property "Footprint" "Capacitor_SMD:C_0603_1608Metric"
 			(at 136.8552 234.95 0)
 			(effects
@@
 			)
 		)
-		(property "Footprint" ""
+		(property "Footprint" "Capacitor_SMD:C_0603_1608Metric"
 			(at 147.32 67.31 0)
 			(effects
@@
 			)
 		)
-		(property "Footprint" "A_HDJ_Library:CP_Elec_6.3x7.7"
+		(property "Footprint" "Capacitor_SMD:CP_Elec_6.3x7.7"
 			(at 435.3052 262.89 0)
 			(effects
@@
 			)
 		)
-		(property "Footprint" "A_HDJ_Library:CP_Elec_6.3x7.7"
+		(property "Footprint" "Capacitor_SMD:CP_Elec_6.3x7.7"
 			(at 130.5052 256.54 0)
 			(effects
@@
 			)
 		)
-		(property "Footprint" "A_HDJ_Library:C_0402_1005Metric"
+		(property "Footprint" "Capacitor_SMD:C_0603_1608Metric"
 			(at 425.1452 262.89 0)
 			(effects
@@
 			)
 		)
-		(property "Footprint" "A_HDJ_Library:CP_Elec_6.3x7.7"
+		(property "Footprint" "Capacitor_SMD:CP_Elec_6.3x7.7"
 			(at 465.7852 262.89 0)
 			(effects
@@
 			)
 		)
-		(property "Footprint" "A_HDJ_Library:CP_Elec_6.3x7.7"
+		(property "Footprint" "Capacitor_SMD:CP_Elec_6.3x7.7"
 			(at 125.4252 256.54 0)
 			(effects
@@
 			)
 		)
-		(property "Footprint" ""
+		(property "Footprint" "Capacitor_SMD:C_0603_1608Metric"
 			(at 147.32 71.12 0)
 			(effects
@@
 			)
 		)
-		(property "Footprint" ""
+		(property "Footprint" "Capacitor_SMD:C_0603_1608Metric"
 			(at 443.23 73.66 0)
 			(effects
@@
 			)
 		)
-		(property "Footprint" ""
+		(property "Footprint" "Capacitor_SMD:C_0603_1608Metric"
 			(at 443.23 81.28 0)
 			(effects
@@
 			)
 		)
-		(property "Footprint" "A_HDJ_Library:C_0402_1005Metric"
+		(property "Footprint" "Capacitor_SMD:C_0603_1608Metric"
 			(at 141.9352 234.95 0)
 			(effects
@@
 			)
 		)
-		(property "Footprint" "A_HDJ_Library:C_0402_1005Metric"
+		(property "Footprint" "Capacitor_SMD:C_0603_1608Metric"
 			(at 120.3452 256.54 0)
 			(effects

Commit message: Lots of tiny capacitors
Parts:
- C139, C140, C143, C147, C148, C149, C151, C152, C155, C158, C159, C161: footprint Capacitor_SMD:C_0603_1608Metric -> Capacitor_SMD:C_0402_1005Metric
Changed lines of the file:
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@@
 			)
 		)
-		(property "Footprint" "Capacitor_SMD:C_0603_1608Metric"
+		(property "Footprint" "Capacitor_SMD:C_0402_1005Metric"
 			(at 155.9052 256.54 0)
 			(effects
@@
 			)
 		)
-		(property "Footprint" "Capacitor_SMD:C_0603_1608Metric"
+		(property "Footprint" "Capacitor_SMD:C_0402_1005Metric"
 			(at 460.7052 262.89 0)
 			(effects
@@
 			)
 		)
-		(property "Footprint" "Capacitor_SMD:C_0603_1608Metric"
+		(property "Footprint" "Capacitor_SMD:C_0402_1005Metric"
 			(at 420.0652 262.89 0)
 			(effects
@@
 			)
 		)
-		(property "Footprint" "Capacitor_SMD:C_0603_1608Metric"
+		(property "Footprint" "Capacitor_SMD:C_0402_1005Metric"
 			(at 441.6552 241.3 0)
 			(effects
@@
 			)
 		)
-		(property "Footprint" "Capacitor_SMD:C_0603_1608Metric"
+		(property "Footprint" "Capacitor_SMD:C_0402_1005Metric"
 			(at 147.32 74.93 0)
 			(effects
@@
 			)
 		)
-		(property "Footprint" "Capacitor_SMD:C_0603_1608Metric"
+		(property "Footprint" "Capacitor_SMD:C_0402_1005Metric"
 			(at 443.23 77.47 0)
 			(effects
@@
 			)
 		)
-		(property "Footprint" "Capacitor_SMD:C_0603_1608Metric"
+		(property "Footprint" "Capacitor_SMD:C_0402_1005Metric"
 			(at 115.2652 256.54 0)
 			(effects
@@
 			)
 		)
-		(property "Footprint" "Capacitor_SMD:C_0603_1608Metric"
+		(property "Footprint" "Capacitor_SMD:C_0402_1005Metric"
 			(at 136.8552 234.95 0)
 			(effects
@@
 			)
 		)
-		(property "Footprint" "Capacitor_SMD:C_0603_1608Metric"
+		(property "Footprint" "Capacitor_SMD:C_0402_1005Metric"
 			(at 425.1452 262.89 0)
 			(effects
@@
 			)
 		)
-		(property "Footprint" "Capacitor_SMD:C_0603_1608Metric"
+		(property "Footprint" "Capacitor_SMD:C_0402_1005Metric"
 			(at 147.32 71.12 0)
 			(effects
@@
 			)
 		)
-		(property "Footprint" "Capacitor_SMD:C_0603_1608Metric"
+		(property "Footprint" "Capacitor_SMD:C_0402_1005Metric"
 			(at 443.23 81.28 0)
 			(effects
@@
 			)
 		)
-		(property "Footprint" "Capacitor_SMD:C_0603_1608Metric"
+		(property "Footprint" "Capacitor_SMD:C_0402_1005Metric"
 			(at 120.3452 256.54 0)
 			(effects

Commit message: Add most passive component footprints
Parts:
- R104, R105, R106, R107: footprint (none) -> Resistor_SMD:R_0402_1005Metric
Changed lines of the file:
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@@
 			)
 		)
-		(property "Footprint" ""
+		(property "Footprint" "Resistor_SMD:R_0402_1005Metric"
 			(at 171.45 113.03 0)
 			(effects
@@
 			)
 		)
-		(property "Footprint" ""
+		(property "Footprint" "Resistor_SMD:R_0402_1005Metric"
 			(at 467.36 119.38 0)
 			(effects
@@
 			)
 		)
-		(property "Footprint" ""
+		(property "Footprint" "Resistor_SMD:R_0402_1005Metric"
 			(at 171.45 110.49 0)
 			(effects
@@
 			)
 		)
-		(property "Footprint" ""
+		(property "Footprint" "Resistor_SMD:R_0402_1005Metric"
 			(at 467.36 116.84 0)
 			(effects

Commit message: Add m.2 slot footprints
Parts:
- added H6, H8: MountingHole, symbol Mechanical:MountingHole
- J7, J8: footprint (none) -> EasyEDA2KiCAD:CONN-SMD_AS0BC21-S48BE-7H
Changed lines of the file:
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@@
+	)
+	(symbol
+		(lib_id "Mechanical:MountingHole")
+		(at 121.92 77.47 0)
+		(unit 1)
+		(exclude_from_sim no)
+		(in_bom no)
+		(on_board yes)
+		(dnp no)
+		(fields_autoplaced yes)
+		(property "Reference" "H6"
+			(at 124.46 76.1999 0)
+			(effects
+				(font
+					(size 1.27 1.27)
+				)
+				(justify left)
+			)
+		)
+		(property "Value" "MountingHole"
+			(at 124.46 78.7399 0)
+			(effects
+				(font
+					(size 1.27 1.27)
+				)
+				(justify left)
+			)
+		)
+		(property "Footprint" ""
+			(at 121.92 77.47 0)
+			(effects
+				(font
+					(size 1.27 1.27)
+				)
+				(hide yes)
+			)
+		)
+		(property "Datasheet" "~"
+			(at 121.92 77.47 0)
+			(effects
+				(font
+					(size 1.27 1.27)
+				)
+				(hide yes)
+			)
+		)
+		(property "Description" "Mounting Hole without connection"
+			(at 121.92 77.47 0)
+			(effects
+				(font
+					(size 1.27 1.27)
+				)
+				(hide yes)
+			)
+		)
+		(instances
+			(project ""
+				(path "/49abeb3a-c598-45a3-ba6b-595eb04f17a8/9d5e3449-f80a-40f7-badf-e98b58cab83b"
+					(reference "H6")
+					(unit 1)
+				)
+			)
+		)
 	)
 	(symbol
@@
 			)
 		)
-		(property "Footprint" ""
+		(property "Footprint" "EasyEDA2KiCAD:CONN-SMD_AS0BC21-S48BE-7H"
 			(at 436.88 107.95 0)
 			(effects
@@
 			)
 		)
-		(property "Footprint" ""
+		(property "Footprint" "EasyEDA2KiCAD:CONN-SMD_AS0BC21-S48BE-7H"
 			(at 140.97 101.6 0)
 			(effects
@@
 					(unit 1)
 				)
+			)
+		)
+	)
+	(symbol
+		(lib_id "Mechanical:MountingHole")
+		(at 419.1 83.82 0)
+		(unit 1)
+		(exclude_from_sim no)
+		(in_bom no)
+		(on_board yes)
+		(dnp no)
+		(fields_autoplaced yes)
+		(property "Reference" "H8"
+			(at 421.64 82.5499 0)
+			(effects
+				(font
+					(size 1.27 1.27)
+				)
+				(justify left)
+			)
+		)
+		(property "Value" "MountingHole"
+			(at 421.64 85.0899 0)
+			(effects
+				(font
+					(size 1.27 1.27)
+				)
+				(justify left)
+			)
+		)
+		(property "Footprint" ""
+			(at 419.1 83.82 0)
+			(effects
+				(font
+					(size 1.27 1.27)
+				)
+				(hide yes)
+			)
+		)
+		(property "Datasheet" "~"
+			(at 419.1 83.82 0)
+			(effects
+				(font
+					(size 1.27 1.27)
+				)
+				(hide yes)
+			)
+		)
+		(property "Description" "Mounting Hole without connection"
+			(at 419.1 83.82 0)
+			(effects
+				(font
+					(size 1.27 1.27)
+				)
+				(hide yes)
+			)
+		)
+		(instances
+			(project ""
+				(path "/49abeb3a-c598-45a3-ba6b-595eb04f17a8/9d5e3449-f80a-40f7-badf-e98b58cab83b"
+					(reference "H8")
+					(unit 1)
+				)

Commit message: Finish fixing footprints
Parts:
- removed H6, H8: MountingHole, symbol Mechanical:MountingHole
- removed J8: Bus_M.2_Socket_E, EasyEDA2KiCAD:CONN-SMD_AS0BC21-S48BE-7H, symbol Connector:Bus_M.2_Socket_E
- added H5, H6: MountingHole_Pad, MountingHole:MountingHole_2.2mm_M2_Pad_Via, symbol Mechanical:MountingHole_Pad
- added J7: Bus_M.2_Socket_E, EasyEDA2KiCAD:CONN-SMD_AS0BC21-S48BE-7H, symbol Connector:Bus_M.2_Socket_E
- renumbered C145 to C139, C146 to C140, C156 to C141, C147 to C142, C157 to C143, C148 to C144, C158 to C145, C159 to C146, C143 to C147, C144 to C148, C155 to C149, C160 to C150, C139 to C151, C140 to C152, C141 to C153, C142 to C154, C149 to C155, C150 to C156, C151 to C157, C152 to C158, C153 to C159, C154 to C160, J7 to J6, J6 to J8
Connections:
- net +3V3: now also J7.2 (3.3V), J7.4 (3.3V), J7.72 (3.3V), J7.74 (3.3V)
- net GND: now also J6.MP, H5.1, H6.1, J7.1 (GND), J7.18 (GND), J7.33 (GND), J7.39 (GND), J7.45 (GND), J7.51 (GND), J7.53 (~{CLKREQ0}), J7.57 (GND), J7.63 (GND), J7.69 (GND), J7.7 (GND), J7.75 (GND), J7.MP
- net SLOT3_M2E.REFCLK+: now also J7.47 (REFCLKp0)
- net SLOT3_M2E.REFCLK-: now also J7.49 (REFCLKn0)
- net SLOT3_M2E.Rx0+: now also J7.41 (PERp0)
- net SLOT3_M2E.Rx0-: now also J7.43 (PERn0)
- net SLOT3_M2E.SUSCLK: now also J7.50 (SUSCLK)
- net SLOT3_M2E.Tx0+: now also J7.35 (PETp0)
- net SLOT3_M2E.Tx0-: now also J7.37 (PETn0)
- net SLOT3_M2E.USB-D+: now also J7.3 (USB_D+)
- net SLOT3_M2E.USB-D-: now also J7.5 (USB_D-)
- net SLOT3_M2E.~{PLTRST}: now also J7.52 (~{PERST0})
- net SLOT3_M2E.~{WAKE}: now also J7.55 (~{PEWAKE0})
- net at R107.1: now also J7.54 (~{W_DISABLE2})
- net at R106.1: now also J7.56 (~{W_DISABLE1})
