File: KiCad/nvme.kicad_sch (KiCad schematic)
At the start: 40 parts, among them J10 Bus_M.2_Socket_M, J11 Bus_M.2_Socket_M, J12 Bus_M.2_Socket_M, J13 Bus_M.2_Socket_M, J14 Bus_M.2_Socket_M

Commit message: Start moving components to module sheets to save sheets
Parts:
- removed C163, C164, C165, C166, C167, C168, C175, C176, C177, C178: 10uF, Capacitor_SMD:C_0603_1608Metric, symbol Device:C_Small
- removed C169, C170, C171, C172, C173, C174, C179, C180, C181, C182: 100nF, Capacitor_SMD:C_0402_1005Metric, symbol Device:C_Small
- removed D22, D23, D24, D25, D26: LED, LED_SMD:LED_0603_1608Metric, symbol Device:LED
- removed H10, H11, H7, H8, H9: MountingHole_Pad, MountingHole:MountingHole_2.2mm_M2_Pad_Via, symbol Mechanical:MountingHole_Pad
- removed J10, J11, J12, J13, J14: Bus_M.2_Socket_M, EasyEDA2KiCAD:CONN-SMD_AS0BC21-S30BM-7H, symbol Connector:Bus_M.2_Socket_M
- removed R108, R109, R110, R111, R112: 2.2k, Resistor_SMD:R_0402_1005Metric, symbol Device:R_Small
- added J10, J11, J12: SFF-8654-8i, EasyEDA2KiCAD:CONN-SMD_HBH2-74AT-1-UHR, symbol Custom:SFF-8654-8i
Connections:
- new net: J10.A1 (GND), J10.A10 (GND), J10.A13 (GND), J10.A16 (GND), J10.A19 (GND), J10.A4 (GND), J10.A7 (GND), J10.B1 (GND), J10.B10 (GND), J10.B13 (GND), J10.B16 (GND), J10.B19 (GND), J10.B4 (GND), J10.B7 (GND)
- new net: J12.A1 (GND), J12.A10 (GND), J12.A13 (GND), J12.A16 (GND), J12.A19 (GND), J12.A4 (GND), J12.A7 (GND), J12.B1 (GND), J12.B10 (GND), J12.B13 (GND), J12.B16 (GND), J12.B19 (GND), J12.B4 (GND), J12.B7 (GND)
- new net: J11.A1 (GND), J11.A10 (GND), J11.A13 (GND), J11.A16 (GND), J11.A19 (GND), J11.A4 (GND), J11.A7 (GND), J11.B1 (GND), J11.B10 (GND), J11.B13 (GND), J11.B16 (GND), J11.B19 (GND), J11.B4 (GND), J11.B7 (GND)
- new net: J12.A22 (GND), J12.A25 (GND), J12.A28 (GND), J12.A31 (GND), J12.A34 (GND), J12.A37 (GND), J12.B22 (GND), J12.B25 (GND), J12.B28 (GND), J12.B31 (GND), J12.B34 (GND), J12.B37 (GND)
- new net: J10.A22 (GND), J10.A25 (GND), J10.A28 (GND), J10.A31 (GND), J10.A34 (GND), J10.A37 (GND), J10.B22 (GND), J10.B25 (GND), J10.B28 (GND), J10.B31 (GND), J10.B34 (GND), J10.B37 (GND)
- new net: J11.A22 (GND), J11.A25 (GND), J11.A28 (GND), J11.A31 (GND), J11.A34 (GND), J11.A37 (GND), J11.B22 (GND), J11.B25 (GND), J11.B28 (GND), J11.B31 (GND), J11.B34 (GND), J11.B37 (GND)
- new net SLOT1_NVMEA.REFCLK+: J10.A11 (REFCLKA+)
- new net SLOT1_NVMEA.REFCLK-: J10.A12 (REFCLKA-)
- new net SLOT1_NVMEA.Rx0+: J10.A2 (PERp0)
- new net SLOT1_NVMEA.Rx0-: J10.A3 (PERn0)
- new net SLOT1_NVMEA.~{WAKE}: J10.A9 (CWAKEA#)
- no-connect marks 55 -> 0
