File: KiCad/psu.kicad_sch (KiCad schematic)
At the start: 20 parts, among them J1 ATX-24, J2 Conn_02x04_Top_Bottom, U6 TPS54331

Commit message: Re-annotate schematic
Parts:
- renumbered C130 to C132, C131 to C133, C132 to C134, C133 to C135, C134 to C136, C135 to C137, C136 to C138, C137 to C139, C138 to C140, R99 to R92, R100 to R93, R101 to R94, R102 to R95, R103 to R96
Changed lines of the file:
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@@
 		(dnp no)
 		(fields_autoplaced yes)
-		(property "Reference" "#PWR0111"
+		(property "Reference" "#PWR0109"
 			(at 58.42 109.22 0)
 			(effects
@@
 			(project ""
 				(path "/49abeb3a-c598-45a3-ba6b-595eb04f17a8/73807de7-58af-4eca-b212-2dba82ac67f9"
-					(reference "#PWR0111")
+					(reference "#PWR0109")
 					(unit 1)
 				)
@@
 		(on_board yes)
 		(dnp no)
-		(property "Reference" "C135"
+		(property "Reference" "C137"
 			(at 148.844 85.852 0)
 			(effects
@@
 			(project "LattePandaMuCluster"
 				(path "/49abeb3a-c598-45a3-ba6b-595eb04f17a8/73807de7-58af-4eca-b212-2dba82ac67f9"
-					(reference "C135")
+					(reference "C137")
 					(unit 1)
 				)
@@
 		(dnp no)
 		(fields_autoplaced yes)
-		(property "Reference" "#PWR0104"
+		(property "Reference" "#PWR0102"
 			(at 179.07 83.82 0)
 			(effects
@@
 			(project ""
 				(path "/49abeb3a-c598-45a3-ba6b-595eb04f17a8/73807de7-58af-4eca-b212-2dba82ac67f9"
-					(reference "#PWR0104")
+					(reference "#PWR0102")
 					(unit 1)
 				)
@@
 		(dnp no)
 		(fields_autoplaced yes)
-		(property "Reference" "C130"
+		(property "Reference" "C132"
 			(at 127.0063 73.66 90)
 			(effects
@@
 			(project ""
 				(path "/49abeb3a-c598-45a3-ba6b-595eb04f17a8/73807de7-58af-4eca-b212-2dba82ac67f9"
-					(reference "C130")
+					(reference "C132")
 					(unit 1)
 				)
@@
 		(on_board yes)
 		(dnp no)
-		(property "Reference" "R100"
+		(property "Reference" "R93"
 			(at 94.234 83.82 0)
 			(effects
@@
 			(project ""
 				(path "/49abeb3a-c598-45a3-ba6b-595eb04f17a8/73807de7-58af-4eca-b212-2dba82ac67f9"
-					(reference "R100")
+					(reference "R93")
 					(unit 1)
 				)
@@
 		(dnp no)
 		(fields_autoplaced yes)
-		(property "Reference" "#PWR0110"
+		(property "Reference" "#PWR0108"
 			(at 97.79 110.49 0)
 			(effects
@@
 			(project ""
 				(path "/49abeb3a-c598-45a3-ba6b-595eb04f17a8/73807de7-58af-4eca-b212-2dba82ac67f9"
-					(reference "#PWR0110")
+					(reference "#PWR0108")
 					(unit 1)
 				)
@@
 		(on_board yes)
 		(dnp no)
-		(property "Reference" "C136"
+		(property "Reference" "C138"
 			(at 96.266 91.948 90)
 			(effects
@@
 			(project ""
 				(path "/49abeb3a-c598-45a3-ba6b-595eb04f17a8/73807de7-58af-4eca-b212-2dba82ac67f9"
-					(reference "C136")
+					(reference "C138")
 					(unit 1)
 				)
@@
 		(dnp no)
 		(fields_autoplaced yes)
-		(property "Reference" "#PWR0100"
+		(property "Reference" "#PWR098"
 			(at 73.66 63.5 0)
 			(effects
@@
 			(project ""
 				(path "/49abeb3a-c598-45a3-ba6b-595eb04f17a8/73807de7-58af-4eca-b212-2dba82ac67f9"
-					(reference "#PWR0100")
+					(reference "#PWR098")
 					(unit 1)
 				)
@@
 		(on_board yes)
 		(dnp no)
-		(property "Reference" "C138"
+		(property "Reference" "C140"
 			(at 101.346 91.948 90)
 			(effects
@@
 			(project "LattePandaMuCluster"
 				(path "/49abeb3a-c598-45a3-ba6b-595eb04f17a8/73807de7-58af-4eca-b212-2dba82ac67f9"
-					(reference "C138")
+					(reference "C140")
 					(unit 1)
 				)
@@
 		(on_board yes)
 		(dnp no)
-		(property "Reference" "C131"
+		(property "Reference" "C133"
 			(at 79.502 84.582 90)
 			(effects
@@
 			(project "LattePandaMuCluster"
 				(path "/49abeb3a-c598-45a3-ba6b-595eb04f17a8/73807de7-58af-4eca-b212-2dba82ac67f9"
-					(reference "C131")
+					(reference "C133")
 					(unit 1)
 				)
@@
 		(dnp no)
 		(fields_autoplaced yes)
-		(property "Reference" "#PWR0103"
+		(property "Reference" "#PWR0101"
 			(at 179.07 67.31 0)
 			(effects
@@
 			(project ""
 				(path "/49abeb3a-c598-45a3-ba6b-595eb04f17a8/73807de7-58af-4eca-b212-2dba82ac67f9"
-					(reference "#PWR0103")
+					(reference "#PWR0101")
 					(unit 1)
 				)
@@
 		(on_board yes)
 		(dnp no)
-		(property "Reference" "C134"
+		(property "Reference" "C136"
 			(at 142.494 85.852 0)
 			(effects
@@
 			(project ""
 				(path "/49abeb3a-c598-45a3-ba6b-595eb04f17a8/73807de7-58af-4eca-b212-2dba82ac67f9"
-					(reference "C134")
+					(reference "C136")
 					(unit 1)
 				)
@@
 		(dnp no)
 		(fields_autoplaced yes)
-		(property "Reference" "#PWR0107"
+		(property "Reference" "#PWR0105"
 			(at 83.82 97.79 0)
 			(effects
@@
 			(project ""
 				(path "/49abeb3a-c598-45a3-ba6b-595eb04f17a8/73807de7-58af-4eca-b212-2dba82ac67f9"
-					(reference "#PWR0107")
+					(reference "#PWR0105")
 					(unit 1)
 				)
@@
 		(dnp no)
 		(fields_autoplaced yes)
-		(property "Reference" "#PWR0102"
+		(property "Reference" "#PWR0100"
 			(at 85.09 63.5 0)
 			(effects
@@
 			(project ""
 				(path "/49abeb3a-c598-45a3-ba6b-595eb04f17a8/73807de7-58af-4eca-b212-2dba82ac67f9"
-					(reference "#PWR0102")
+					(reference "#PWR0100")
 					(unit 1)
 				)
@@
 		(on_board yes)
 		(dnp no)
-		(property "Reference" "R101"
+		(property "Reference" "R94"
 			(at 134.62 85.852 90)
 			(effects
@@
 			(project ""
 				(path "/49abeb3a-c598-45a3-ba6b-595eb04f17a8/73807de7-58af-4eca-b212-2dba82ac67f9"
-					(reference "R101")
+					(reference "R94")
 					(unit 1)
 				)
@@
 		(on_board yes)
 		(dnp no)
-		(property "Reference" "#PWR0108"
+		(property "Reference" "#PWR0106"
 			(at 111.76 100.33 0)
 			(effects
@@
 			(project ""
 				(path "/49abeb3a-c598-45a3-ba6b-595eb04f17a8/73807de7-58af-4eca-b212-2dba82ac67f9"
-					(reference "#PWR0108")
+					(reference "#PWR0106")
 					(unit 1)
 				)
@@
 		(dnp no)
 		(fields_autoplaced yes)
-		(property "Reference" "#PWR0106"
+		(property "Reference" "#PWR0104"
 			(at 52.07 90.17 0)
 			(effects
@@
 			(project ""
 				(path "/49abeb3a-c598-45a3-ba6b-595eb04f17a8/73807de7-58af-4eca-b212-2dba82ac67f9"
-					(reference "#PWR0106")
+					(reference "#PWR0104")
 					(unit 1)
 				)
@@
 		(on_board yes)
 		(dnp no)
-		(property "Reference" "R102"
+		(property "Reference" "R95"
 			(at 128.524 88.9 0)
 			(effects
@@
 			(project ""
 				(path "/49abeb3a-c598-45a3-ba6b-595eb04f17a8/73807de7-58af-4eca-b212-2dba82ac67f9"
-					(reference "R102")
+					(reference "R95")
 					(unit 1)
 				)
@@
 		(on_board yes)
 		(dnp no)
-		(property "Reference" "R99"
+		(property "Reference" "R92"
 			(at 89.916 81.026 90)
 			(effects
@@
 			(project ""
 				(path "/49abeb3a-c598-45a3-ba6b-595eb04f17a8/73807de7-58af-4eca-b212-2dba82ac67f9"
-					(reference "R99")
+					(reference "R92")
 					(unit 1)
 				)
@@
 		(on_board yes)
 		(dnp no)
-		(property "Reference" "#PWR0109"
+		(property "Reference" "#PWR0107"
 			(at 124.46 102.87 0)
 			(effects
@@
 			(project ""
 				(path "/49abeb3a-c598-45a3-ba6b-595eb04f17a8/73807de7-58af-4eca-b212-2dba82ac67f9"
-					(reference "#PWR0109")
+					(reference "#PWR0107")
 					(unit 1)
 				)
@@
 		(on_board yes)
 		(dnp no)
-		(property "Reference" "C133"
+		(property "Reference" "C135"
 			(at 84.582 84.582 90)
 			(effects
@@
 			(project ""
 				(path "/49abeb3a-c598-45a3-ba6b-595eb04f17a8/73807de7-58af-4eca-b212-2dba82ac67f9"
-					(reference "C133")
+					(reference "C135")
 					(unit 1)
 				)
@@
 		(on_board yes)
 		(dnp no)
-		(property "Reference" "R103"
+		(property "Reference" "R96"
 			(at 100.584 100.076 0)
 			(effects
@@
 			(project ""
 				(path "/49abeb3a-c598-45a3-ba6b-595eb04f17a8/73807de7-58af-4eca-b212-2dba82ac67f9"
-					(reference "R103")
+					(reference "R96")
 					(unit 1)
 				)
@@
 		(dnp no)
 		(fields_autoplaced yes)
-		(property "Reference" "#PWR0101"
+		(property "Reference" "#PWR099"
 			(at 78.74 63.5 0)
 			(effects
@@
 			(project ""
 				(path "/49abeb3a-c598-45a3-ba6b-595eb04f17a8/73807de7-58af-4eca-b212-2dba82ac67f9"
-					(reference "#PWR0101")
+					(reference "#PWR099")
 					(unit 1)
 				)
@@
 		(dnp no)
 		(fields_autoplaced yes)
-		(property "Reference" "#PWR099"
+		(property "Reference" "#PWR097"
 			(at 68.58 63.5 0)
 			(effects
@@
 			(project ""
 				(path "/49abeb3a-c598-45a3-ba6b-595eb04f17a8/73807de7-58af-4eca-b212-2dba82ac67f9"
-					(reference "#PWR099")
+					(reference "#PWR097")
 					(unit 1)
 				)
@@
 		(on_board yes)
 		(dnp no)
-		(property "Reference" "C132"
+		(property "Reference" "C134"
 			(at 82.042 84.582 90)
 			(effects
@@
 			(project "LattePandaMuCluster"
 				(path "/49abeb3a-c598-45a3-ba6b-595eb04f17a8/73807de7-58af-4eca-b212-2dba82ac67f9"
-					(reference "C132")
+					(reference "C134")
 					(unit 1)
 				)
@@
 		(on_board yes)
 		(dnp no)
-		(property "Reference" "#PWR0105"
+		(property "Reference" "#PWR0103"
 			(at 148.59 86.36 0)
 			(effects
@@
 			(project "LattePandaMuCluster"
 				(path "/49abeb3a-c598-45a3-ba6b-595eb04f17a8/73807de7-58af-4eca-b212-2dba82ac67f9"
-					(reference "#PWR0105")
+					(reference "#PWR0103")
 					(unit 1)
 				)
@@
 		(dnp no)
 		(fields_autoplaced yes)
-		(property "Reference" "#PWR0112"
+		(property "Reference" "#PWR0110"
 			(at 40.64 121.92 0)
 			(effects
@@
 			(project ""
 				(path "/49abeb3a-c598-45a3-ba6b-595eb04f17a8/73807de7-58af-4eca-b212-2dba82ac67f9"
-					(reference "#PWR0112")
+					(reference "#PWR0110")
 					(unit 1)
 				)
@@
 		(on_board yes)
 		(dnp no)
-		(property "Reference" "C137"
+		(property "Reference" "C139"
 			(at 98.806 91.948 90)
 			(effects
@@
 			(project ""
 				(path "/49abeb3a-c598-45a3-ba6b-595eb04f17a8/73807de7-58af-4eca-b212-2dba82ac67f9"
-					(reference "C137")
-					(unit 1)
-				)
+					(reference "C139")
+					(unit 1)
+				)
