File: KiCad/stm32.kicad_sch (KiCad schematic)
At the start: 18 parts, among them J15 Conn_02x05_Odd_Even, J16 Conn_02x05_Odd_Even, U7 STM32F030C8Tx, Y1 25MHz

Commit message: Re-annotate schematic
Parts:
- renumbered C183 to C193, C184 to C194, C185 to C195, C186 to C196, C187 to C197, C188 to C198, C189 to C199, C191 to C200, C190 to C201, C192 to C202, J15 to J16, J16 to J17, R113 to R106, R114 to R107, R115 to R108
Changed lines of the file:
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@@
 		(on_board yes)
 		(dnp no)
-		(property "Reference" "C187"
+		(property "Reference" "C197"
 			(at 109.474 78.74 90)
 			(effects
@@
 			(project ""
 				(path "/49abeb3a-c598-45a3-ba6b-595eb04f17a8/6eac886f-f669-4a66-b218-dbac55577930"
-					(reference "C187")
+					(reference "C197")
 					(unit 1)
 				)
@@
 		(on_board yes)
 		(dnp no)
-		(property "Reference" "C186"
+		(property "Reference" "C196"
 			(at 131.064 76.2 90)
 			(effects
@@
 			(project "LattePandaMuCluster"
 				(path "/49abeb3a-c598-45a3-ba6b-595eb04f17a8/6eac886f-f669-4a66-b218-dbac55577930"
-					(reference "C186")
+					(reference "C196")
 					(unit 1)
 				)
@@
 		(on_board yes)
 		(dnp no)
-		(property "Reference" "C184"
+		(property "Reference" "C194"
 			(at 109.474 73.66 90)
 			(effects
@@
 			(project "LattePandaMuCluster"
 				(path "/49abeb3a-c598-45a3-ba6b-595eb04f17a8/6eac886f-f669-4a66-b218-dbac55577930"
-					(reference "C184")
+					(reference "C194")
 					(unit 1)
 				)
@@
 		(on_board yes)
 		(dnp no)
-		(property "Reference" "#PWR0177"
+		(property "Reference" "#PWR0185"
 			(at 78.74 111.76 0)
 			(effects
@@
 			(project "LattePandaMuCluster"
 				(path "/49abeb3a-c598-45a3-ba6b-595eb04f17a8/6eac886f-f669-4a66-b218-dbac55577930"
-					(reference "#PWR0177")
+					(reference "#PWR0185")
 					(unit 1)
 				)
@@
 		(dnp no)
 		(fields_autoplaced yes)
-		(property "Reference" "R115"
+		(property "Reference" "R108"
 			(at 101.6 88.9 90)
 			(effects
@@
 			(project ""
 				(path "/49abeb3a-c598-45a3-ba6b-595eb04f17a8/6eac886f-f669-4a66-b218-dbac55577930"
-					(reference "R115")
+					(reference "R108")
 					(unit 1)
 				)
@@
 		(dnp no)
 		(fields_autoplaced yes)
-		(property "Reference" "J15"
+		(property "Reference" "J16"
 			(at 184.15 80.01 0)
 			(effects
@@
 			(project ""
 				(path "/49abeb3a-c598-45a3-ba6b-595eb04f17a8/6eac886f-f669-4a66-b218-dbac55577930"
-					(reference "J15")
+					(reference "J16")
 					(unit 1)
 				)
@@
 		(on_board yes)
 		(dnp no)
-		(property "Reference" "#PWR0176"
+		(property "Reference" "#PWR0184"
 			(at 97.79 110.49 0)
 			(effects
@@
 			(project "LattePandaMuCluster"
 				(path "/49abeb3a-c598-45a3-ba6b-595eb04f17a8/6eac886f-f669-4a66-b218-dbac55577930"
-					(reference "#PWR0176")
+					(reference "#PWR0184")
 					(unit 1)
 				)
@@
 		(on_board yes)
 		(dnp no)
-		(property "Reference" "C188"
+		(property "Reference" "C198"
 			(at 131.064 78.74 90)
 			(effects
@@
 			(project "LattePandaMuCluster"
 				(path "/49abeb3a-c598-45a3-ba6b-595eb04f17a8/6eac886f-f669-4a66-b218-dbac55577930"
-					(reference "C188")
+					(reference "C198")
 					(unit 1)
 				)
@@
 		(on_board yes)
 		(dnp no)
-		(property "Reference" "C192"
+		(property "Reference" "C202"
 			(at 85.344 106.934 90)
 			(effects
@@
 			(project "LattePandaMuCluster"
 				(path "/49abeb3a-c598-45a3-ba6b-595eb04f17a8/6eac886f-f669-4a66-b218-dbac55577930"
-					(reference "C192")
+					(reference "C202")
 					(unit 1)
 				)
@@
 		(on_board yes)
 		(dnp no)
-		(property "Reference" "#PWR0175"
+		(property "Reference" "#PWR0181"
 			(at 160.02 101.6 0)
 			(effects
@@
 			(project ""
 				(path "/49abeb3a-c598-45a3-ba6b-595eb04f17a8/6eac886f-f669-4a66-b218-dbac55577930"
-					(reference "#PWR0175")
+					(reference "#PWR0181")
 					(unit 1)
 				)
@@
 		(on_board yes)
 		(dnp no)
-		(property "Reference" "#PWR0178"
+		(property "Reference" "#PWR0186"
 			(at 149.86 109.22 0)
 			(effects
@@
 			(project ""
 				(path "/49abeb3a-c598-45a3-ba6b-595eb04f17a8/6eac886f-f669-4a66-b218-dbac55577930"
-					(reference "#PWR0178")
+					(reference "#PWR0186")
 					(unit 1)
 				)
@@
 		(on_board yes)
 		(dnp no)
-		(property "Reference" "C185"
+		(property "Reference" "C195"
 			(at 109.474 76.2 90)
 			(effects
@@
 			(project "LattePandaMuCluster"
 				(path "/49abeb3a-c598-45a3-ba6b-595eb04f17a8/6eac886f-f669-4a66-b218-dbac55577930"
-					(reference "C185")
+					(reference "C195")
 					(unit 1)
 				)
@@
 		(on_board yes)
 		(dnp no)
-		(property "Reference" "C189"
+		(property "Reference" "C199"
 			(at 154.432 92.964 90)
 			(effects
@@
 			(project ""
 				(path "/49abeb3a-c598-45a3-ba6b-595eb04f17a8/6eac886f-f669-4a66-b218-dbac55577930"
-					(reference "C189")
+					(reference "C199")
 					(unit 1)
 				)
@@
 		(on_board yes)
 		(dnp no)
-		(property "Reference" "#PWR0354"
+		(property "Reference" "#PWR0182"
 			(at 193.04 101.6 0)
 			(effects
@@
 			(project ""
 				(path "/49abeb3a-c598-45a3-ba6b-595eb04f17a8/6eac886f-f669-4a66-b218-dbac55577930"
-					(reference "#PWR0354")
+					(reference "#PWR0182")
 					(unit 1)
 				)
@@
 		(dnp no)
 		(fields_autoplaced yes)
-		(property "Reference" "#PWR0171"
+		(property "Reference" "#PWR0177"
 			(at 184.15 76.2 0)
 			(effects
@@
 			(project ""
 				(path "/49abeb3a-c598-45a3-ba6b-595eb04f17a8/6eac886f-f669-4a66-b218-dbac55577930"
-					(reference "#PWR0171")
+					(reference "#PWR0177")
 					(unit 1)
 				)
@@
 		(dnp no)
 		(fields_autoplaced yes)
-		(property "Reference" "#PWR0180"
+		(property "Reference" "#PWR0188"
 			(at 120.65 176.53 0)
 			(effects
@@
 			(project ""
 				(path "/49abeb3a-c598-45a3-ba6b-595eb04f17a8/6eac886f-f669-4a66-b218-dbac55577930"
-					(reference "#PWR0180")
+					(reference "#PWR0188")
 					(unit 1)
 				)
@@
 		(dnp no)
 		(fields_autoplaced yes)
-		(property "Reference" "#PWR0174"
+		(property "Reference" "#PWR0180"
 			(at 91.44 93.98 0)
 			(effects
@@
 			(project ""
 				(path "/49abeb3a-c598-45a3-ba6b-595eb04f17a8/6eac886f-f669-4a66-b218-dbac55577930"
-					(reference "#PWR0174")
+					(reference "#PWR0180")
 					(unit 1)
 				)
@@
 		(on_board yes)
 		(dnp no)
-		(property "Reference" "#PWR0355"
+		(property "Reference" "#PWR0183"
 			(at 180.34 96.52 0)
 			(effects
@@
 			(project "LattePandaMuCluster"
 				(path "/49abeb3a-c598-45a3-ba6b-595eb04f17a8/6eac886f-f669-4a66-b218-dbac55577930"
-					(reference "#PWR0355")
+					(reference "#PWR0183")
 					(unit 1)
 				)
@@
 		(on_board yes)
 		(dnp no)
-		(property "Reference" "C183"
+		(property "Reference" "C193"
 			(at 109.474 71.12 90)
 			(effects
@@
 			(project "LattePandaMuCluster"
 				(path "/49abeb3a-c598-45a3-ba6b-595eb04f17a8/6eac886f-f669-4a66-b218-dbac55577930"
-					(reference "C183")
+					(reference "C193")
 					(unit 1)
 				)
@@
 		(on_board yes)
 		(dnp no)
-		(property "Reference" "C191"
+		(property "Reference" "C200"
 			(at 193.548 92.964 90)
 			(effects
@@
 			(project "LattePandaMuCluster"
 				(path "/49abeb3a-c598-45a3-ba6b-595eb04f17a8/6eac886f-f669-4a66-b218-dbac55577930"
-					(reference "C191")
+					(reference "C200")
 					(unit 1)
 				)
@@
 		(on_board yes)
 		(dnp no)
-		(property "Reference" "R113"
+		(property "Reference" "R106"
 			(at 173.228 74.93 0)
 			(effects
@@
 			(project "LattePandaMuCluster"
 				(path "/49abeb3a-c598-45a3-ba6b-595eb04f17a8/6eac886f-f669-4a66-b218-dbac55577930"
-					(reference "R113")
+					(reference "R106")
 					(unit 1)
 				)
@@
 		(on_board yes)
 		(dnp no)
-		(property "Reference" "R114"
+		(property "Reference" "R107"
 			(at 190.754 74.93 0)
 			(effects
@@
 			(project ""
 				(path "/49abeb3a-c598-45a3-ba6b-595eb04f17a8/6eac886f-f669-4a66-b218-dbac55577930"
-					(reference "R114")
+					(reference "R107")
 					(unit 1)
 				)
@@
 		(on_board yes)
 		(dnp no)
-		(property "Reference" "#PWR0173"
+		(property "Reference" "#PWR0179"
 			(at 138.43 87.63 0)
 			(effects
@@
 			(project "LattePandaMuCluster"
 				(path "/49abeb3a-c598-45a3-ba6b-595eb04f17a8/6eac886f-f669-4a66-b218-dbac55577930"
-					(reference "#PWR0173")
+					(reference "#PWR0179")
 					(unit 1)
 				)
@@
 		(on_board yes)
 		(dnp no)
-		(property "Reference" "#PWR0172"
+		(property "Reference" "#PWR0178"
 			(at 104.14 87.63 0)
 			(effects
@@
 			(project ""
 				(path "/49abeb3a-c598-45a3-ba6b-595eb04f17a8/6eac886f-f669-4a66-b218-dbac55577930"
-					(reference "#PWR0172")
+					(reference "#PWR0178")
 					(unit 1)
 				)
@@
 		(on_board yes)
 		(dnp no)
-		(property "Reference" "#PWR0179"
+		(property "Reference" "#PWR0187"
 			(at 171.45 111.76 0)
 			(effects
@@
 			(project ""
 				(path "/49abeb3a-c598-45a3-ba6b-595eb04f17a8/6eac886f-f669-4a66-b218-dbac55577930"
-					(reference "#PWR0179")
+					(reference "#PWR0187")
 					(unit 1)
 				)
@@
 		(on_board yes)
 		(dnp no)
-		(property "Reference" "C190"
+		(property "Reference" "C201"
 			(at 84.328 98.044 90)
 			(effects
@@
 			(project "LattePandaMuCluster"
 				(path "/49abeb3a-c598-45a3-ba6b-595eb04f17a8/6eac886f-f669-4a66-b218-dbac55577930"
-					(reference "C190")
+					(reference "C201")
 					(unit 1)
 				)
@@
 		(dnp no)
 		(fields_autoplaced yes)
-		(property "Reference" "#PWR0170"
+		(property "Reference" "#PWR0176"
 			(at 118.11 66.04 0)
 			(effects
@@
 			(project ""
 				(path "/49abeb3a-c598-45a3-ba6b-595eb04f17a8/6eac886f-f669-4a66-b218-dbac55577930"
-					(reference "#PWR0170")
+					(reference "#PWR0176")
 					(unit 1)
 				)
@@
 		(on_board yes)
 		(dnp no)
-		(property "Reference" "J16"
+		(property "Reference" "J17"
 			(at 154.94 106.68 0)
 			(effects
@@
 			(project "LattePandaMuCluster"
 				(path "/49abeb3a-c598-45a3-ba6b-595eb04f17a8/6eac886f-f669-4a66-b218-dbac55577930"
-					(reference "J16")
-					(unit 1)
-				)
+					(reference "J17")
+					(unit 1)
+				)
